File: hardware/kicad/crypto_node.kicad_sch (KiCad schematic)
At the start: 0 parts

Commit message: nothing
Parts:
- added R28, R31, R32, R33: 0Ω, symbol Device:R
Connections:
- net GPS/GPS_RX: now also R28.2
- net GPS/GPS_TX: now also R31.2
- net LoRA/LORA_RX: now also R32.2
- net LoRA/LORA_TX: now also R33.2
- new net STM32/USART1_RX: R33.1
- new net STM32/USART1_TX: R32.1
- new net STM32/USART2_RX: R31.1
- new net STM32/USART2_TX: R28.1
Other:
- sheet LoRA ports: added LORA_M0, LORA_M1; removed none
- sheet STM32 ports: added ADC1_IN6, PB14, PB15; removed BATTERY_PERCENTAGE

Commit message: finished schematics
Other:
- sheet Tampering renamed Tamper
- sheet STM32 ports: added PC13; removed none
- sheet Tamper ports: added TAMPER; removed none
Changed lines of the file:
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@@
-	(wire
-		(pts
-			(xy 99.06 88.9) (xy 121.92 88.9)
-		)
-		(stroke
-			(width 0)
-			(type default)
-		)
-	)
 	(wire
 		(pts
@@
 	(wire
 		(pts
+			(xy 162.56 38.1) (xy 154.94 38.1)
+		)
+		(stroke
+			(width 0)
+			(type default)
+		)
+	)
+	(wire
+		(pts
+			(xy 99.06 91.44) (xy 121.92 91.44)
+		)
+		(stroke
+			(width 0)
+			(type default)
+		)
+	)
+	(wire
+		(pts
 			(xy 175.26 91.44) (xy 182.88 91.44)
 		)
@@
 	(wire
 		(pts
+			(xy 154.94 38.1) (xy 154.94 73.66)
+		)
+		(stroke
+			(width 0)
+			(type default)
+		)
+	)
+	(wire
+		(pts
 			(xy 152.4 114.3) (xy 152.4 120.65)
 		)
@@
 	(wire
 		(pts
+			(xy 99.06 86.36) (xy 121.92 86.36)
+		)
+		(stroke
+			(width 0)
+			(type default)
+		)
+	)
+	(wire
+		(pts
 			(xy 152.4 128.27) (xy 152.4 135.89)
 		)
@@
 		(pts
 			(xy 142.24 38.1) (xy 142.24 73.66)
-		)
-		(stroke
-			(width 0)
-			(type default)
-		)
-	)
-	(wire
-		(pts
-			(xy 99.06 92.71) (xy 121.92 92.71)
 		)
 		(stroke
@@
 		)
 		(pin "I2C1_SCL" output
-			(at 121.92 88.9 180)
+			(at 121.92 86.36 180)
 			(effects
 				(font
@@
 		)
 		(pin "I2C1_SDA" bidirectional
-			(at 121.92 92.71 180)
+			(at 121.92 91.44 180)
 			(effects
 				(font
@@
 			)
 		)
-		(pin "PB14" passive
+		(pin "PB14" output
 			(at 175.26 104.14 0)
 			(effects
@@
 			)
 		)
-		(pin "PB15" passive
+		(pin "PB15" output
 			(at 175.26 100.33 0)
+			(effects
+				(font
+					(size 1.27 1.27)
+				)
+				(justify right)
+			)
+		)
+		(pin "PC13" input
+			(at 154.94 73.66 90)
 			(effects
 				(font
@@
 		)
 		(pin "CRYPT_SCL" input
-			(at 99.06 88.9 0)
+			(at 99.06 86.36 0)
 			(effects
 				(font
@@
 		)
 		(pin "CRYPT_SDA" bidirectional
-			(at 99.06 92.71 0)
+			(at 99.06 91.44 0)
 			(effects
 				(font
@@
 			(color 0 0 0 0)
 		)
-		(property "Sheetname" "Tampering"
+		(property "Sheetname" "Tamper"
 			(at 162.56 19.6084 0)
 			(show_name no)
@@
 			)
 		)
+		(pin "TAMPER" output
+			(at 162.56 38.1 180)
+			(effects
+				(font
+					(size 1.27 1.27)
+				)
+				(justify left)
+			)
+		)

Commit message: schematics refinement
Parts:
- R1: renamed from R28; footprint (none) -> Resistor_SMD:R_0805_2012Metric_Pad1.20x1.40mm_HandSolder
- R2: renamed from R31; footprint (none) -> Resistor_SMD:R_0805_2012Metric_Pad1.20x1.40mm_HandSolder
- R3: renamed from R32; footprint (none) -> Resistor_SMD:R_0805_2012Metric_Pad1.20x1.40mm_HandSolder
- R4: renamed from R33; footprint (none) -> Resistor_SMD:R_0805_2012Metric_Pad1.20x1.40mm_HandSolder
Other:
- sheet LoRA ports: added AUX; removed none
- sheet Power ports: added POWER_VOLTAGE; removed BATTERY_PERCENTAGE
- sheet STM32 ports: added PB5; removed none
Changed lines of the file:
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@@
+	(wire
+		(pts
+			(xy 175.26 107.95) (xy 198.12 107.95)
+		)
+		(stroke
+			(width 0)
+			(type default)
+		)
+	)
 	(wire
 		(pts
@@
 		(in_pos_files yes)
 		(dnp no)
-		(property "Reference" "R32"
+		(property "Reference" "R3"
 			(at 186.69 86.36 90)
 			(show_name no)
@@
 			)
 		)
-		(property "Footprint" ""
+		(property "Footprint" "Resistor_SMD:R_0805_2012Metric_Pad1.20x1.40mm_HandSolder"
 			(at 186.69 88.138 90)
 			(hide yes)
@@
 			(project "crypto_node"
 				(path "/6c72b0cb-17b9-42a6-811c-297d0c354af3"
-					(reference "R32")
+					(reference "R3")
 					(unit 1)
 				)
@@
 		(in_pos_files yes)
 		(dnp no)
-		(property "Reference" "R33"
+		(property "Reference" "R4"
 			(at 186.69 91.44 90)
 			(show_name no)
@@
 			)
 		)
-		(property "Footprint" ""
+		(property "Footprint" "Resistor_SMD:R_0805_2012Metric_Pad1.20x1.40mm_HandSolder"
 			(at 186.69 93.218 90)
 			(hide yes)
@@
 			(project "crypto_node"
 				(path "/6c72b0cb-17b9-42a6-811c-297d0c354af3"
-					(reference "R33")
+					(reference "R4")
 					(unit 1)
 				)
@@
 		(in_pos_files yes)
 		(dnp no)
-		(property "Reference" "R31"
+		(property "Reference" "R2"
 			(at 153.67 123.19 0)
 			(show_name no)
@@
 			)
 		)
-		(property "Footprint" ""
+		(property "Footprint" "Resistor_SMD:R_0805_2012Metric_Pad1.20x1.40mm_HandSolder"
 			(at 150.622 124.46 90)
 			(hide yes)
@@
 			(project "crypto_node"
 				(path "/6c72b0cb-17b9-42a6-811c-297d0c354af3"
-					(reference "R31")
+					(reference "R2")
 					(unit 1)
 				)
@@
 		(in_pos_files yes)
 		(dnp no)
-		(property "Reference" "R28"
+		(property "Reference" "R1"
 			(at 147.32 123.19 0)
 			(show_name no)
@@
 			)
 		)
-		(property "Footprint" ""
+		(property "Footprint" "Resistor_SMD:R_0805_2012Metric_Pad1.20x1.40mm_HandSolder"
 			(at 144.272 124.46 90)
 			(hide yes)
@@
 			(project "crypto_node"
 				(path "/6c72b0cb-17b9-42a6-811c-297d0c354af3"
-					(reference "R28")
+					(reference "R1")
 					(unit 1)
 				)
@@
 			)
 		)
-		(pin "BATTERY_PERCENTAGE" output
+		(pin "POWER_VOLTAGE" output
 			(at 134.62 38.1 0)
 			(effects
@@
 		(pin "PC13" input
 			(at 154.94 73.66 90)
+			(effects
+				(font
+					(size 1.27 1.27)
+				)
+				(justify right)
+			)
+		)
+		(pin "PB5" input
+			(at 175.26 107.95 0)
 			(effects
 				(font
@@
 			(effects
 				(font
+					(size 1.27 1.27)
+				)
+				(justify left)
+			)
+		)
+		(pin "AUX" output
+			(at 198.12 107.95 180)
+			(effects
+				(font

Commit message: started PCB and changed power system
Parts:
- added H1, H2, H3, H4: Mount_Hole, MountingHole:MountingHole_3.2mm_M3_Pad_Via, symbol Mechanical:MountingHole_Pad
Connections:
- new net GND: H1.1, H2.1, H3.1, H4.1
Other:
- sheet Power ports: added BATTERY_VOLTAGE; removed POWER_VOLTAGE
- note added: "MOUNTING HOLES"
