File: hardware/kicad/Power.kicad_sch (KiCad schematic)
At the start: 0 parts

Commit message: boost converter
Parts:
- added BT1: 103450 Li-PO, symbol Device:Battery_Cell
- added C1, C2: μF, symbol Device:C
- added C3, C7: 100nF, symbol Device:C
- added C4: 10μF, symbol Device:C
- added C5, C6: 22μF, symbol Device:C
- added L1: 1μH, symbol Device:L
- added R1, R2, R3, R4: Ω, symbol Device:R
- added R5: 1KΩ, symbol Device:R
- added R6: 732KΩ, symbol Device:R
- added R7: 100KΩ, symbol Device:R
- added U1: (no value), Package_TO_SOT_SMD:SOT-563, symbol TPS61023DRLR:TPS61023DRLR
Connections:
- new net +5V: C5.1, C6.1, C7.1, R6.1, U1.6 (VOUT)
- new net +BATT: BT1.1 (+), R3.1
- new net +VCOM: C3.1, C4.1, L1.1, R5.1, U1.3 (VIN)
- new net GND: BT1.2 (-), C3.2, C4.2, C5.2, C6.2, C7.2, R4.2, R7.2, U1.4 (GND)
- new net TPS_EN: R5.2, U1.2 (EN)
- new net TPS_FB: R6.2, R7.1, U1.1 (FB)
- new net TPS_SW: L1.2, U1.5 (SW)
- new net battery_charge: R3.2, R4.1
Other:
- note added: "BATTERY"
- note added: "BUCK CONVERTER (3V7 -> 5V 3A MAX)"

Commit message: done power
Parts:
- added C10, C13, C14, C15, C18, C19: 10μF, symbol Device:C
- added C11, C12, C16, C17, C20, C9: 100nF, symbol Device:C
- added D1: 1SMA4734A, symbol Device:D_Zener
- added D2: LED, symbol Device:LED
- added Q1: FDN304PZ, PCM_SparkFun-Semiconductor-Standard:SOT23-3, symbol PCM_SparkFun-DiscreteSemi:Q_PMOS_4.2A_20V
- added R8: 100KΩ, symbol Device:R
- added R9: KΩ, symbol Device:R
- added SW1: SW_SPDT_321, symbol Switch:SW_SPDT_321
- added U2, U3, U4: TLV74333PDBVR, Package_TO_SOT_SMD:SOT-23-5_HandSoldering, symbol TLV74333PDBVR:TLV74333PDBVR
Connections:
- net +5V: now also C10.1, C11.1, C14.1, C17.1, C18.1, C9.1, U2.1 (VIN), U2.3 (EN), U3.1 (VIN), U3.3 (EN), U4.1 (VIN), U4.3 (EN)
- net +BATT: now also Q1.3 (D)
- net +VCOM: now also R9.1, SW1.3 (A)
- net GND: now also C10.2, C11.2, C12.2, C13.2, C14.2, C15.2, C16.2, C17.2, C18.2, C19.2, C20.2, C9.2, D2.1 (K), R8.1, U2.2 (GND), U3.2 (GND), U4.2 (GND)
- new net: C15.1, C16.1, U3.5 (OUT)
- new net +BATT_POLA: D1.1 (K), Q1.2 (S), SW1.2 (B)
- new net +GPS_3V3: C19.1, C20.1, U4.5 (OUT)
- new net +STM_3V3: C12.1, C13.1, U2.5 (OUT)
- new net INDI_LED: D2.2 (A), R9.2
- new net PMOS_GATE: D1.2 (A), Q1.1 (G), R8.2
- no-connect marks 0 -> 1
Other:
- note added: "BATTERY (1S Li-Po)"
- note added: "CRYPT LDO"
- note added: "GPS LDO"
- note added: "POLARITY PROTECTION AND SWITCHING"
- note added: "STM32 LDO"
- note removed: "BATTERY"

Commit message: done power
Connections:
- net +CRYPT_3V3: now also C15.1, C16.1, U3.5 (OUT)
Changed lines of the file:
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@@
 		(at 128.27 46.99)
-	)
-	(bus_entry
-		(at 165.1 153.67)
-		(size 2.54 2.54)
-		(stroke
-			(width 0)
-			(type default)
-		)
 	)
 	(wire
@@
 					(unit 1)
 				)
+			)
+		)
+	)
+	(symbol
+		(lib_id "power:VPP")
+		(at 276.86 68.58 0)
+		(unit 1)
+		(body_style 1)
+		(exclude_from_sim no)
+		(in_bom yes)
+		(on_board yes)
+		(in_pos_files yes)
+		(dnp no)
+		(property "Reference" "#PWR037"
+			(at 276.86 72.39 0)
+			(hide yes)
+			(show_name no)
+			(do_not_autoplace no)
+			(effects
+				(font
+					(size 1.27 1.27)
+				)
+			)
+		)
+		(property "Value" "+CRYPT_3V3"
+			(at 276.86 64.77 0)
+			(show_name no)
+			(do_not_autoplace no)
+			(effects
+				(font
+					(size 1.27 1.27)
+				)
+			)
+		)
+		(property "Footprint" ""
+			(at 276.86 68.58 0)
+			(hide yes)
+			(show_name no)
+			(do_not_autoplace no)
+			(effects
+				(font
+					(size 1.27 1.27)
+				)
+			)
+		)
+		(property "Datasheet" ""
+			(at 276.86 68.58 0)
+			(hide yes)
+			(show_name no)
+			(do_not_autoplace no)
+			(effects
+				(font
+					(size 1.27 1.27)
+				)
+			)
+		)
+		(property "Description" "Power symbol creates a global label with name \"VPP\""
+			(at 276.86 68.58 0)
+			(hide yes)
+			(show_name no)
+			(do_not_autoplace no)
+			(effects
+				(font
+					(size 1.27 1.27)
+				)
+			)
+		)
+		(pin "1"
+		)
+		(instances
+			(project "crypto_node"
+				(path "/6c72b0cb-17b9-42a6-811c-297d0c354af3/0878dbd6-f23a-45b7-803f-70f55a38d748"
+					(reference "#PWR037")
+					(unit 1)
+				)

Commit message: power completed
Parts:
- removed D2: LED, symbol Device:LED
- added C32, C41, C42, C43: 10μF, symbol Device:C
- added C40: 100nf, symbol Device:C
- added D2: SLESD5Z5C, Diode_SMD:D_SOD-523, symbol SLESD5Z5C:SLESD5Z5C
- added D7, D8, D9: white, LED_SMD:LED_0603_1608Metric, symbol Device:LED
- added J19: USB_C_Receptacle_USB2.0_16P, Connector_USB:USB_C_Receptacle_GCT_USB4105-xx-A_16P_TopMnt_Horizontal, symbol Connector:USB_C_Receptacle_USB2.0_16P
- added R15, R16: 5K1Ω, symbol Device:R
- added R17, R18, R19: 470Ω, symbol Device:R
- added R23: 100KΩ, symbol Device:R
- added R24, R27: 10KΩ, symbol Device:R
- added R25: 33KΩ, symbol Device:R
- added R26: 3K3Ω, symbol Device:R
- added U6: MCP73871-2CC, Package_DFN_QFN:QFN-20-1EP_4x4mm_P0.5mm_EP2.5x2.5mm, symbol Battery_Management:MCP73871-2CC
- C17, C18, C19, C20, U4: now not fitted; now left out of the parts list
- R9: value KΩ -> 270KΩ
Connections:
- net +VCOM: now also C43.1, U6.1 (OUT), U6.20 (OUT); no longer R9.1, SW1.3 (A)
- net GND: now also C32.2, C40.2, C41.2, C42.2, C43.2, D2.1, J19.A1 (GND), J19.A12 (GND), J19.B1 (GND), J19.B12 (GND), J19.S1 (SHIELD), R15.2, R16.2, R23.2, R24.2, R25.2, R26.2, U6.10 (V_{SS}), U6.11 (V_{SS}), U6.21 (V_{SS})
- net INDI_LED renamed VPCC
- net VPCC: now also R23.1, U6.2 (VPCC)
- net battery_charge renamed BATTERY_PERCENTAGE
- new net: D9.1 (K), R17.2
- new net: D7.1 (K), R18.2
- new net: D8.1 (K), R19.2
- new net +BATT_PROC: C42.1, SW1.3 (A), U6.14 (V_{BAT}), U6.15 (V_{BAT}), U6.16 (V_{BAT_SENSE})
- new net +VUSB: C32.1, C40.1, C41.1, D2.2, D7.2 (A), D8.2 (A), D9.2 (A), J19.A4 (VBUS), J19.A9 (VBUS), J19.B4 (VBUS), J19.B9 (VBUS), R27.1, R9.1, U6.18 (IN), U6.19 (IN)
- new net CC1: J19.A5 (CC1), R15.1
- new net CC2: J19.B5 (CC2), R16.1
- new net CE: R27.2, U6.17 (CE), U6.3 (SEL), U6.4 (PROG2), U6.9 (~{TE})
- new net PROG1: R26.1, U6.13 (PROG1)
- new net PROG3: R25.1, U6.12 (PROG3)
- new net STAT2: R19.1, U6.7 (STAT2)
- new net THERM: R24.1, U6.5 (THERM)
- new net ~{LBO}: R18.1, U6.8 (STAT1/~{LBO})
- new net ~{PG}: R17.1, U6.6 (~{PG})
- no-connect marks 1 -> 29
Other:
- note added: "BOOST CONVERTER (3V7 -> 5V 1.5A MAX)"
- note added: "CHARGING AND TEMPERA RESISTOR"
- note added: "CONFIG PINS"
- note added: "DECOUPLING CAPACITORS"
- note added: "DECOUPLING CAPS"
- note added: "LED INDICATORS"
- note added: "MCP73871 (POWER DISTRIBUTION AND Li-Po CHARGER)"
- note added: "SURGE PROTECTION"
- note added: "USB (POWER ONLY)"
- note removed: "BUCK CONVERTER (3V7 -> 5V 3A MAX)"
- moved on the sheet: C3, C4, C5, C6, C7, D1, L1, Q1, R3, R4, R5, R6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

Commit message: tweeks
Parts:
- R3, R4: value Ω -> 10KΩ
Connections:
- net +VUSB: now also U6.17 (CE), U6.3 (SEL), U6.4 (PROG2), U6.9 (~{TE})
- net GND: now also R27.2
- removed net CE: R27.2, U6.17 (CE), U6.3 (SEL), U6.4 (PROG2), U6.9 (~{TE})
