File: hardware/kicad/Power.kicad_sch (KiCad schematic)
At the start: 36 parts, among them J2 USB_C_Receptacle_USB2.0_16P, Q1 FDN304PZ, SW1 SW_SPDT_321, U1 TPS563201, U2 TLV74333PDBVR, U3 TLV74333PDBVR

Commit message: Final hardware cleanup push (hopefully)
Other:
- company: (none) -> Done By :- Arudhran
- title: (none) -> Cryptographic Tactical Node
