File: hardware/kicad/STM32.kicad_sch (KiCad schematic)
At the start: 0 parts

Commit message: power completed
Parts:
- added C21, C8: μF, symbol Device:C
- added C22: 4μ7F, symbol Device:C
- added C23, C30: 10μF, symbol Device:C
- added C24, C25, C26, C27, C28, C29, C33, C38: 100nF, symbol Device:C
- added C31: 18pF, symbol Device:C
- added C34: 33pF, symbol Device:C
- added C35: 27pF, symbol Device:C
- added C36: 11pF, symbol Device:C
- added C37: 15pF, symbol Device:C
- added C39: 22pF, symbol Device:C
- added D5: white, LED_SMD:LED_0603_1608Metric, symbol Device:LED
- added D6: WS2812B-2020, LED_SMD:LED_WS2812B-2020_PLCC4_2.0x2.0mm, symbol LED:WS2812B-2020
- added FB1: BLM18AG121SN1D, Inductor_SMD:L_0603_1608Metric, symbol Device:FerriteBead
- added J5: 01x06_Pin, Connector_PinHeader_2.54mm:PinHeader_1x06_P2.54mm_Vertical, symbol Connector:Conn_01x06_Pin
- added JP2, JP3, JP4: Jumper, Jumper:SolderJumper-2_P1.3mm_Open_RoundedPad1.0x1.5mm, symbol Jumper:SolderJumper_2_Open
- added R10, R11: Ω, symbol Device:R
- added R12, R13, R14: 10KΩ, symbol Device:R
- added R20: 470Ω, symbol Device:R
- added R21: 4K7Ω, symbol Device:R
- added R22: 2K2Ω, symbol Device:R
- added S1, S2: TSA017A2518B, TSA017A2518B:TSA017A2518B, symbol dk_Tactile-Switches:B3F-1000
- added U5: STM32F411CEUx, Package_DFN_QFN:QFN-48-1EP_7x7mm_P0.5mm_EP5.6x5.6mm, symbol MCU_ST_STM32F4:STM32F411CEUx
- added Y1: YSX321SL-25MHz, Crystal:Crystal_SMD_3225-4Pin_3.2x2.5mm, symbol Device:Crystal_GND24
- added Y2: YXC-Y-26, Crystal:Crystal_DS26_D2.0mm_L6.0mm_Horizontal, symbol Device:Crystal
Connections:
- new net: J5.2 (Pin_2), JP3.2 (B)
- new net: J5.6 (Pin_6), JP2.2 (B)
- new net +STM_3V3: C23.1, C24.1, C25.1, C26.1, C27.1, C28.1, C30.1, D6.4 (VDD), FB1.1, JP2.1 (A), JP4.2 (B), R13.1, R21.1, R22.1, S2.3, S2.4, U5.1 (VBAT), U5.24 (VDD), U5.36 (VDD), U5.48 (VDD)
- new net +STM_3V3_A: C29.1, FB1.2, U5.9 (VDDA)
- new net BOOT0: C33.1, R14.1, S2.1, S2.2, U5.44 (BOOT0)
- new net BOOT1: JP4.1 (A), R12.1, U5.20 (PB2)
- new net GND: C22.2, C23.2, C24.2, C25.2, C26.2, C27.2, C28.2, C29.2, C30.2, C31.2, C33.2, C34.2, C36.2, C38.2, C39.2, D5.1 (K), D6.2 (VSS), J5.4 (Pin_4), R12.2, R14.2, S1.3, S1.4, U5.23 (VSS), U5.35 (VSS), U5.47 (VSS), U5.49 (VSS), U5.8 (VSSA), Y1.2, Y1.4
- new net I2C1_SCL: R21.2, U5.45 (PB8)
- new net I2C1_SDA: R22.2, U5.46 (PB9)
- new net NRST: C38.1, JP3.1 (A), R13.2, S1.1, S1.2, U5.7 (NRST)
- new net PROG_LED: D6.3 (DIN)
- new net RCC_OSC32_IN: C39.1, U5.3 (PC14), Y1.1
- new net RCC_OSC32_OUT: C34.1, U5.4 (PC15), Y1.3
- new net RCC_OSC_IN: U5.5 (PH0)
- new net RCC_OSC_OUT: C31.1, C36.1, U5.6 (PH1), Y2.1, Y2.2
- new net STATUS_LED: R20.1
- new net STM_LED: D5.2 (A), R20.2
- new net SYS_JTCK-SWCLK: J5.5 (Pin_5), U5.37 (PA14)
- new net SYS_JTDO-SWO: J5.1 (Pin_1), U5.39 (PB3)
- new net SYS_JTMS-SWDIO: J5.3 (Pin_3), U5.34 (PA13)
- new net USART1_RX: U5.31 (PA10)
- new net USART1_TX: U5.30 (PA9)
- new net USART2_RX: U5.13 (PA3)
- new net USART2_TX: U5.12 (PA2)
- new net VCAP_1: C22.1, U5.22 (VCAP1)
- no-connect marks 0 -> 13
Other:
- note added: "ANALOG FILTERING"
- note added: "BOOT TACTILE SWITCH"
- note added: "BOOT1 SELECTOR"
- note added: "BUILT-IN LED"
- note added: "DECOUPLING CAPS"
- note added: "HSE CRYSTAL"
- note added: "I2C PULL-UP"
- note added: "LSE CRYSTAL"
- note added: "PROGRAMABLE RGB LED"
- note added: "RESET TACTILE SWITCH"
- note added: "ST-LINK DEBUGGER AND FLASHING"

Commit message: tweeks
Connections:
- net RCC_OSC32_IN: now also C31.1, Y2.2; no longer C39.1, Y1.1
- net RCC_OSC32_OUT: now also C36.1, Y2.1; no longer C34.1, Y1.3
- net RCC_OSC_IN: now also C39.1, Y1.1
- net RCC_OSC_OUT: now also C34.1, Y1.3; no longer C31.1, C36.1, Y2.1, Y2.2
Changed lines of the file:
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@@
 		)
 	)
-	(global_label "RCC_OSC_OUT"
-		(shape input)
-		(at 64.77 99.06 90)
-		(effects
-			(font
-				(size 1.27 1.27)
-			)
-			(justify left)
-		)
-		(property "Intersheetrefs" "${INTERSHEET_REFS}"
-			(at 64.77 99.06 90)
+	(global_label "RCC_OSC_IN"
+		(shape input)
+		(at 39.37 99.06 90)
+		(effects
+			(font
+				(size 1.27 1.27)
+			)
+			(justify left)
+		)
+		(property "Intersheetrefs" "${INTERSHEET_REFS}"
+			(at 39.37 99.06 90)
 			(hide yes)
 			(show_name no)
@@
 	(global_label "RCC_OSC_OUT"
 		(shape input)
+		(at 19.05 99.06 90)
+		(effects
+			(font
+				(size 1.27 1.27)
+			)
+			(justify left)
+		)
+		(property "Intersheetrefs" "${INTERSHEET_REFS}"
+			(at 19.05 99.06 90)
+			(hide yes)
+			(show_name no)
+			(do_not_autoplace no)
+			(effects
+				(font
+					(size 1.27 1.27)
+				)
+			)
+		)
+	)
+	(global_label "RCC_OSC32_OUT"
+		(shape input)
+		(at 64.77 99.06 90)
+		(effects
+			(font
+				(size 1.27 1.27)
+			)
+			(justify left)
+		)
+		(property "Intersheetrefs" "${INTERSHEET_REFS}"
+			(at 64.77 99.06 90)
+			(hide yes)
+			(show_name no)
+			(do_not_autoplace no)
+			(effects
+				(font
+					(size 1.27 1.27)
+				)
+			)
+		)
+	)
+	(global_label "STATUS_LED"
+		(shape input)
+		(at 97.79 109.22 180)
+		(fields_autoplaced yes)
+		(effects
+			(font
+				(size 1.27 1.27)
+			)
+			(justify right)
+		)
+		(property "Intersheetrefs" "${INTERSHEET_REFS}"
+			(at 83.6168 109.22 0)
+			(hide yes)
+			(show_name no)
+			(do_not_autoplace no)
+			(effects
+				(font
+					(size 1.27 1.27)
+				)
+				(justify right)
+			)
+		)
+	)
+	(global_label "RCC_OSC32_IN"
+		(shape input)
 		(at 49.53 99.06 90)
 		(effects
@@
 			(hide yes)
 			(show_name no)
-			(do_not_autoplace no)
-			(effects
-				(font
-					(size 1.27 1.27)
-				)
-			)
-		)
-	)
-	(global_label "RCC_OSC32_OUT"
-		(shape input)
-		(at 19.05 99.06 90)
-		(effects
-			(font
-				(size 1.27 1.27)
-			)
-			(justify left)
-		)
-		(property "Intersheetrefs" "${INTERSHEET_REFS}"
-			(at 19.05 99.06 90)
-			(hide yes)
-			(show_name no)
-			(do_not_autoplace no)
-			(effects
-				(font
-					(size 1.27 1.27)
-				)
-			)
-		)
-	)
-	(global_label "STATUS_LED"
-		(shape input)
-		(at 97.79 109.22 180)
-		(fields_autoplaced yes)
-		(effects
-			(font
-				(size 1.27 1.27)
-			)
-			(justify right)
-		)
-		(property "Intersheetrefs" "${INTERSHEET_REFS}"
-			(at 83.6168 109.22 0)
-			(hide yes)
-			(show_name no)
-			(do_not_autoplace no)
-			(effects
-				(font
-					(size 1.27 1.27)
-				)
-				(justify right)
-			)
-		)
-	)
-	(global_label "RCC_OSC32_IN"
-		(shape input)
-		(at 39.37 99.06 90)
-		(effects
-			(font
-				(size 1.27 1.27)
-			)
-			(justify left)
-		)
-		(property "Intersheetrefs" "${INTERSHEET_REFS}"
-			(at 39.37 99.06 90)
-			(hide yes)
-			(show_name no)
