File: hardware/kicad/STM32.kicad_sch (KiCad schematic)
At the start: 39 parts, among them J5 01x06_Pin, U5 STM32F411CEUx, Y1 YSX321SL-25MHz, Y2 YXC-Y-26

Commit message: nothing
Connections:
- net PROG_LED: now also U5.19 (PB1)
- net STATUS_LED: now also U5.25 (PB12)
- net ADC1_IN6: now reaches U5.16 (PA6)
- net PB14: now reaches U5.27 (PB14)
- net PB15: now reaches U5.28 (PB15)
- no-connect marks 35 -> 30
Changed lines of the file:
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@@
 	)
 	(no_connect
-		(at 130.81 85.09)
-	)
-	(no_connect
 		(at 130.81 97.79)
 	)
@@
 	)
 	(no_connect
-		(at 130.81 118.11)
-	)
-	(no_connect
 		(at 57.15 87.63)
 	)
@@
 	)
 	(no_connect
-		(at 130.81 115.57)
-	)
-	(no_connect
 		(at 166.37 54.61)
 	)
 	(no_connect
-		(at 166.37 69.85)
-	)
-	(no_connect
-		(at 130.81 110.49)
-	)
-	(no_connect
 		(at 81.28 -15.24)
 	)
@@
 	(wire
 		(pts
+			(xy 123.19 118.11) (xy 130.81 118.11)
+		)
+		(stroke
+			(width 0)
+			(type default)
+		)
+	)
+	(wire
+		(pts
 			(xy 140.97 41.91) (xy 140.97 44.45)
 		)
@@
 	(wire
 		(pts
+			(xy 166.37 69.85) (xy 173.99 69.85)
+		)
+		(stroke
+			(width 0)
+			(type default)
+		)
+	)
+	(wire
+		(pts
 			(xy 241.3 102.87) (xy 246.38 102.87)
 		)
@@
 		)
 	)
+	(wire
+		(pts
+			(xy 123.19 110.49) (xy 130.81 110.49)
+		)
+		(stroke
+			(width 0)
+			(type default)
+		)
+	)
 	(polyline
 		(pts
@@
 	(wire
 		(pts
+			(xy 123.19 115.57) (xy 130.81 115.57)
+		)
+		(stroke
+			(width 0)
+			(type default)
+		)
+	)
+	(wire
+		(pts
 			(xy 38.1 144.78) (xy 38.1 147.32)
 		)
@@
 		)
 	)
+	(wire
+		(pts
+			(xy 123.19 85.09) (xy 130.81 85.09)
+		)
+		(stroke
+			(width 0)
+			(type default)
+		)
+	)
 	(polyline
 		(pts
@@
 	(global_label "PROG_LED"
 		(shape output)
-		(at 97.79 113.03 180)
+		(at 123.19 85.09 180)
 		(fields_autoplaced yes)
 		(effects
@@
 		)
 		(property "Intersheetrefs" "${INTERSHEET_REFS}"
-			(at 85.2496 113.03 0)
+			(at 110.6496 85.09 0)
 			(hide yes)
 			(show_name no)
@@
 	)
 	(global_label "STATUS_LED"
-		(shape input)
-		(at 97.79 109.22 180)
+		(shape output)
+		(at 123.19 110.49 180)
 		(fields_autoplaced yes)
 		(effects
@@
 		)
 		(property "Intersheetrefs" "${INTERSHEET_REFS}"
-			(at 83.6168 109.22 0)
+			(at 109.0168 110.49 0)
 			(hide yes)
 			(show_name no)
@@
 	)
 	(hierarchical_label "I2C1_SCL"
-		(shape passive)
+		(shape output)
 		(at 123.19 102.87 180)
 		(effects
@@
 		)
 	)
-	(hierarchical_label "BATTERY_PERCENTAGE"
-		(shape input)
-		(at 97.79 116.84 180)
+	(hierarchical_label "PB14"
+		(shape passive)
+		(at 123.19 115.57 180)
 		(effects
 			(font
@@
 		)
 	)
-	(hierarchical_label "LORA_CTRL_M0"
-		(shape output)
-		(at 97.79 119.38 180)
+	(hierarchical_label "ADC1_IN6"
+		(shape input)
+		(at 173.99 69.85 0)
+		(effects
+			(font
+				(size 1.27 1.27)
+			)
+			(justify left)
+		)
+	)
+	(hierarchical_label "PB15"
+		(shape passive)
+		(at 123.19 118.11 180)
 		(effects
 			(font
@@
 	)
 	(hierarchical_label "I2C1_SDA"
-		(shape passive)
+		(shape bidirectional)
 		(at 259.08 109.22 0)
 		(effects
@@
 		)
 	)
-	(hierarchical_label "LORA_CRTL_M1"
-		(shape output)
-		(at 97.79 121.92 180)
-		(effects
-			(font
-				(size 1.27 1.27)
-			)
-			(justify right)
-		)
-	)
 	(hierarchical_label "I2C1_SDA"
-		(shape passive)
+		(shape bidirectional)
 		(at 123.19 105.41 180)
 		(effects
@@
 	)
 	(hierarchical_label "I2C1_SCL"
-		(shape passive)
+		(shape output)
 		(at 259.08 102.87 0)
 		(effects
@@
 		)
 		(pin "19"
+			(alternate "TIM3_CH4")
 		)
 		(pin "18"
@@
 		)
 		(pin "16"
+			(alternate "ADC1_IN6")
 		)
 		(pin "15"

Commit message: finished schematics
Parts:
- removed Y1: YSX321SL-25MHz, Crystal:Crystal_SMD_3225-4Pin_3.2x2.5mm, symbol Device:Crystal_GND24
- added Y3: Crystal_GND24, Crystal:Crystal_SMD_3225-4Pin_3.2x2.5mm, symbol Device:Crystal_GND24
- JP2, JP3, JP4: footprint Jumper:SolderJumper-2_P1.3mm_Open_RoundedPad1.0x1.5mm -> Package_TO_SOT_SMD:SOT-23-5_HandSoldering
Connections:
- net +STM_3V3: now also JP2.2 (B); no longer JP2.1 (A)
- net GND: now also Y3.2 (G), Y3.4 (G)
- net NRST: now also JP3.2 (B); no longer JP3.1 (A)
- net RCC_OSC_IN: now also Y3.3
- net RCC_OSC_OUT: now also Y3.1
- net at J5.2 (Pin_2): now also JP3.1 (A); no longer JP3.2 (B)
- net PC13: now reaches U5.2 (PC13)
- net at J5.6 (Pin_6): now also JP2.1 (A); no longer JP2.2 (B)
- no-connect marks 30 -> 29

Commit message: schematics refinement
Parts:
- removed C21, C8: μF, symbol Device:C
- removed R10, R11: Ω, symbol Device:R
- removed R12: 10KΩ, symbol Device:R
- added D8: white, LED_SMD:LED_0805_2012Metric_Pad1.15x1.40mm_HandSolder, symbol Device:LED
- added R27: 470Ω, Resistor_SMD:R_0805_2012Metric_Pad1.20x1.40mm_HandSolder, symbol Device:R
- added R28: 33KΩ, Resistor_SMD:R_0805_2012Metric_Pad1.20x1.40mm_HandSolder, symbol Device:R
- C19: renamed from C34; footprint (none) -> Capacitor_SMD:C_0402_1005Metric_Pad0.74x0.62mm_HandSolder
- C20: renamed from C23; footprint (none) -> Capacitor_SMD:C_1206_3216Metric_Pad1.33x1.80mm_HandSolder
- C21: renamed from C28; footprint (none) -> Capacitor_SMD:C_0603_1608Metric_Pad1.08x0.95mm_HandSolder
- C22: renamed from C35; footprint (none) -> Capacitor_SMD:C_0402_1005Metric_Pad0.74x0.62mm_HandSolder
- C23: renamed from C33; footprint (none) -> Capacitor_SMD:C_0603_1608Metric_Pad1.08x0.95mm_HandSolder
- C24: footprint (none) -> Capacitor_SMD:C_0603_1608Metric_Pad1.08x0.95mm_HandSolder
- C25: renamed from C39; footprint (none) -> Capacitor_SMD:C_0402_1005Metric_Pad0.74x0.62mm_HandSolder
- C26: renamed from C25; footprint (none) -> Capacitor_SMD:C_0603_1608Metric_Pad1.08x0.95mm_HandSolder
- C27: renamed from C38; footprint (none) -> Capacitor_SMD:C_0603_1608Metric_Pad1.08x0.95mm_HandSolder
- C28: renamed from C31; footprint (none) -> Capacitor_SMD:C_0402_1005Metric_Pad0.74x0.62mm_HandSolder
- C29: renamed from C26; footprint (none) -> Capacitor_SMD:C_0603_1608Metric_Pad1.08x0.95mm_HandSolder
- C30: renamed from C29; footprint (none) -> Capacitor_SMD:C_0603_1608Metric_Pad1.08x0.95mm_HandSolder
- C31: renamed from C37; footprint (none) -> Capacitor_SMD:C_0402_1005Metric_Pad0.74x0.62mm_HandSolder
- C32: renamed from C27; footprint (none) -> Capacitor_SMD:C_0603_1608Metric_Pad1.08x0.95mm_HandSolder
- C33: renamed from C36; footprint (none) -> Capacitor_SMD:C_0402_1005Metric_Pad0.74x0.62mm_HandSolder
- C34: renamed from C22; footprint (none) -> Capacitor_SMD:C_0805_2012Metric_Pad1.18x1.45mm_HandSolder
- C35: renamed from C30; footprint (none) -> Capacitor_SMD:C_1206_3216Metric_Pad1.33x1.80mm_HandSolder
- D7: renamed from D5; footprint LED_SMD:LED_0603_1608Metric -> LED_SMD:LED_0805_2012Metric_Pad1.15x1.40mm_HandSolder
- FB1: footprint Inductor_SMD:L_0603_1608Metric -> Inductor_SMD:L_0805_2012Metric_Pad1.05x1.20mm_HandSolder
- JP1: renamed from JP2; footprint Package_TO_SOT_SMD:SOT-23-5_HandSoldering -> Jumper:SolderJumper-2_P1.3mm_Open_RoundedPad1.0x1.5mm
- JP2: renamed from JP3; footprint Package_TO_SOT_SMD:SOT-23-5_HandSoldering -> Jumper:SolderJumper-2_P1.3mm_Open_RoundedPad1.0x1.5mm
- JP3: renamed from JP4; footprint Package_TO_SOT_SMD:SOT-23-5_HandSoldering -> Jumper:SolderJumper-2_P1.3mm_Open_RoundedPad1.0x1.5mm
- R22: renamed from R13; footprint (none) -> Resistor_SMD:R_0805_2012Metric_Pad1.20x1.40mm_HandSolder
- R23: renamed from R14; footprint (none) -> Resistor_SMD:R_0805_2012Metric_Pad1.20x1.40mm_HandSolder
- R24: renamed from R21; footprint (none) -> Resistor_SMD:R_0805_2012Metric_Pad1.20x1.40mm_HandSolder
- R25: renamed from R22; footprint (none) -> Resistor_SMD:R_0805_2012Metric_Pad1.20x1.40mm_HandSolder
- R26: renamed from R20; footprint (none) -> Resistor_SMD:R_0805_2012Metric_Pad1.20x1.40mm_HandSolder
- renumbered J5 to J2, Y3 to Y1
Connections:
- net BOOT1: now also R28.1
- net GND: now also D8.1 (K), R28.2
- net STM_LED: now also D8.2 (A), R27.2
- net STATUS_LED_1: now reaches U5.26 (PB13)
- net STATUS_LED_1: now also R27.1
- net PB5: now reaches U5.41 (PB5)
- net STATUS_LED renamed STATUS_LED_0
- no-connect marks 29 -> 19
Other:
- moved on the sheet: C21, C30, C35, D6, JP3, R24, R25

Commit message: completed schematics and started pcb
Parts:
- Y1: value Crystal_GND24 -> YSX321SL
- Y2: value YXC-Y-26 -> YST310S; footprint Crystal:Crystal_DS26_D2.0mm_L6.0mm_Horizontal -> Crystal:Crystal_SMD_3215-2Pin_3.2x1.5mm
Changed lines of the file:
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@@
 			)
 		)
-		(property "Value" "YXC-Y-26"
+		(property "Value" "YST310S"
 			(at 57.15 106.68 0)
 			(show_name no)
@@
 			)
 		)
-		(property "Footprint" "Crystal:Crystal_DS26_D2.0mm_L6.0mm_Horizontal"
+		(property "Footprint" "Crystal:Crystal_SMD_3215-2Pin_3.2x1.5mm"
 			(at 57.15 110.49 0)
 			(hide yes)
@@
 			)
 		)
-		(property "Value" "Crystal_GND24"
+		(property "Value" "YSX321SL"
 			(at 29.21 105.41 0)
 			(show_name no)
@@
 		)
 	)
-	(group ""
-		(members "0af27c98-53d6-4dd7-97ab-83d67ceb9ae7" "1abd658a-25f1-41a5-a825-8d9e4151692a"
-			"23efd371-966c-4da8-8cfa-ff9e12367358" "263df225-39b4-439a-83ec-af25d9350ee0"
-			"32d92de4-8bbb-4043-9ddf-c00800cc1dc7" "4028dadc-3de0-4ee2-9123-376b616747e1"
-			"406f95b3-de8f-4e4f-9885-4696db3c5a96" "41e44965-719e-44a7-8067-d4f363499bf5"
-			"684dfe04-414b-4bf7-ab3f-996a4f7a1272" "903d4bee-9238-4f64-b2a9-37da136706f6"
-			"93eb9348-a6f0-4cca-88d3-a2c0d8434860" "ad2f5af8-6aa2-428d-826f-8197d62647b6"
-			"c41ad114-47a4-4fa6-a0ea-b320e4760a69" "c9ee1b52-67a0-4b45-8743-843445a7fadf"
-			"cf333c71-07e8-4f2f-a2e7-000a41665e10" "e4c83e2e-51b8-465b-b23e-9cfd735fff09"
-		)
-	)
-	(group ""
-		(members "116eb96b-7e3b-42d0-b5f2-5e39cdd19331" "161e7c61-3cac-4bb5-9e30-4326fef67ece"
-			"182cafd3-2eb3-418d-8802-483ef7121534" "19471f9f-caf5-4454-b940-da7c2fc387de"
-			"211b27f7-1613-4797-8444-bc6b766e29fe" "23e1b050-7649-42f7-9a68-ad773fe6247c"
-			"2887c71e-3a4e-4079-bf92-d8e7b99aa821" "28c5bd13-226e-4d7d-84a7-0e62a160734f"
-			"32b2a22b-9a93-475e-a6dd-e3853d2fca98" "399cab6b-8838-4c0b-8c30-e2cbe967ff94"
-			"3ce65ba1-2a96-4cd6-b4ac-4a602d17666a" "526de933-1ac6-46ed-b997-0642b1f0169e"
-			"533a3b38-c124-4a00-8709-2e9f2b2a22aa" "64566d05-d51b-4197-9a30-5eea1f546428"
-			"657b777b-63db-4ef6-8346-55aa6fb4a1e6" "657e2a14-6000-4849-9330-8a602a9ef762"
-			"6a07439f-50f9-44fe-8fc6-754428290501" "738e5c4d-e87e-439e-a247-5ecef41af8f1"
-			"84649392-2c69-479e-8f3d-b9514b3f544e" "8817ddf1-0d24-4404-bbb9-7b5d8f8d038d"
-			"89007542-0309-486a-a024-95098a304b46" "928a1cff-f509-42b3-a323-3ac6ce2ea033"
-			"9362b5cd-10b9-40c1-906c-af856f7cabad" "94b6158e-188d-4fd1-bd3f-bcc1a2901315"
-			"982479ec-b96a-4b2b-b606-bea4cb6a1ad5" "9f373651-eb58-4515-bfd1-beaa3e70b191"
-			"a2497e9a-44a6-4983-8d9a-5dd73ceb75d2" "a8347aa1-7f88-471d-9db8-dc8e61695a00"
-			"b132d6fe-c2f4-44b9-ba8b-dd748d42d056" "b8d0ed68-1c43-441e-80d1-c0cccc6897b3"
-			"d165934c-7a0f-4753-8dce-84572e5adf2d" "df38b10d-ef9b-4cc3-b729-22d6346c31f6"
-			"e0e76e5a-b261-4ee9-9aa2-7654dc094ad3" "e92b8c21-5fc5-467e-b395-08585c7ba284"
-			"f2fee2c6-b691-45a5-9ff0-8d2aef5135cb" "f3d22b9f-b1ee-4ee1-8469-933ed8e22351"
-			"fe0d2d48-68cc-49e6-b7ac-24cd6a66e282"
-		)
-	)
-	(group ""
-		(members "019968c3-a939-494c-a7db-02a0ee9fce78" "03cca3a1-605f-4ac4-8aa9-95cd9857d214"
-			"05b8e2bc-bdc0-4edc-b756-bc6d5c41e17b" "1fabb93b-4baf-418b-8042-692b4931f778"
-			"21b33e0a-6f77-4c3a-9bf4-ff85e334d535" "24ccf2c2-5f19-4978-940f-98eb598d2474"
-			"290e4a32-0011-4070-af13-0b22f86b10f7" "32ad97d6-a39c-435c-a7e9-360ea7fd2d3a"
-			"3fc264c0-537c-46e4-9dd5-77cfb07503a2" "4199c866-24ac-4f44-9426-5c92b0521b37"
-			"46a0664d-807f-4e22-9bc1-3241f4b926da" "4826441e-85c1-4b17-90b8-a25f4cbf396b"
-			"4910f3ec-88f2-4725-bd76-ec62cde4fdab" "5e0ce231-d36b-46d6-9366-33b06d8b3cc7"
-			"665a8170-91c7-4a87-b6fb-401acaba1458" "6881fd60-0eff-4af4-b346-88480f4c812f"
-			"6ecc3398-5260-4c99-9a9e-d5627ec6f0e1" "749628be-5aa1-4280-98e6-1595ad096441"
-			"9c98a366-1145-45be-9b5b-8b87427bbe2a" "9f0f3f49-bf87-418a-936b-11af4d52c42c"
-			"ac371088-5ff4-420f-846c-68937f06c6f2" "b81b0d01-72f7-411e-b000-3309c25a03f5"
-			"c80b12bf-ea78-4fb9-ad2c-1c1f777d8cd3" "cf5fce77-d9f4-437b-98ad-68c8a235feee"
-			"e0ac7780-58cb-4931-966e-cf51783aa078" "f0f44351-b53e-4b3f-90b2-6930e3f3f339"
-			"f543e436-f211-4936-9902-fdb15fee05cc" "f6a7300f-1806-427b-8e66-a18d89dae570"
-			"fed86a29-199b-467f-b402-ee84673653d8"
-		)
-	)
-	(group ""
-		(members "0912e73c-272b-4ff5-9908-f47402ce7820" "2ca799b8-8cde-4214-902a-a0cc6e8aae5c"
-			"2e4d22b1-9c90-46ff-b5b5-067086059e3b" "3078b53c-f44f-432c-b612-939932e5c4df"
-			"4244ec6c-1cf1-4dda-bb82-45ec8f564574" "4499d93e-9598-4b95-896c-5d097666f11e"
-			"45b212f7-031d-4d08-9fcb-06e7348ef846" "47bc8edb-b1ba-4be5-a2d0-2b8eac8f2590"
-			"51831065-9d83-49d0-a4d8-e25f039ac740" "5ee63311-1c0f-4469-b7ae-a57380224091"
-			"5f8edc5a-a811-4c39-9116-aceba1df3eb0" "6580867c-db1e-4a84-bed4-fe3eb5962224"
-			"684646e0-621c-45cc-9323-bb8fb370aed8" "7a7f3096-f366-4cbe-ab84-c728077cf3e7"
-			"7ac3790d-9254-4e37-b829-52f9a7b1d3b4" "7e9ed2ca-3873-41c3-ac09-b81897ccb7bb"
-			"8e1039ff-b138-4a48-a76e-5da51f5648f9" "99b7789f-7e44-4a35-b7c7-340d738a1940"
-			"acde33b3-a824-40bb-ab49-e97cfa98c049" "b0ba3aee-ffbb-4d42-89f3-2bfd7182a71b"
-			"b3102f68-be6f-4a7d-8e3d-2911287aa6e5" "b699a520-fd5b-477f-99e0-316bf6e48bf5"
-			"d4291e0f-6a94-4ca7-a1da-240fc1ad4ea4" "e4631012-8f65-4c41-82eb-affe7ef3a39d"
-			"e90f5753-5217-4bc5-aea8-08d6d04949b6" "feeca705-764f-4f76-9013-f582650daa4c"
-			"ff295c04-3095-43ff-9db2-7971b81d9ec9"
-		)
-	)
-	(group ""
-		(members "0eeecbae-d947-4c70-a23c-a29aff29ea11" "1a0237ca-6584-497c-a634-1eb40bdcadf4"
-			"2a1f7c13-c194-4637-8063-489a736e57a7" "2f1d5032-b9f8-42f4-8a79-c085c6d0cef7"
-			"3deac820-e0e4-49be-be7d-51548a818948" "573929e8-b0bd-41b5-90ef-f908a64042a5"
-			"6f20a9db-b158-42d2-ad6c-7867a383acdb" "730cc222-5b68-4d19-a4ea-7e545dee2e41"
-			"7affabd4-55ad-4041-9dd2-70e4caae201c" "7b49134f-dfae-4a96-a338-ddd729268ddd"
-			"88db7da6-e472-467f-968a-fee0ea869f37" "a6cb2fb3-5614-40d4-b71a-9d1e40530d40"
-			"bc2f3001-1925-43d2-98c7-b3debf2cc45a" "c5cb9f9b-e9f5-45fd-a7c6-fc144fdddfad"
-			"d6f8657c-4b03-42d2-beab-e457105dc614" "deb2468b-58c0-4c86-a669-69836496ccc7"
-			"edc70b2b-e47c-44ba-96c1-23aff64b0abc"
-		)
-	)

Commit message: started PCB and changed power system
Parts:
- removed C21: 100nF, Capacitor_SMD:C_0603_1608Metric_Pad1.08x0.95mm_HandSolder, symbol Device:C
- removed R24: 4K7Ω, Resistor_SMD:R_0805_2012Metric_Pad1.20x1.40mm_HandSolder, symbol Device:R
- added C31: 100nF, Capacitor_SMD:C_0603_1608Metric_Pad1.08x0.95mm_HandSolder, symbol Device:C
- added R15: 5K1Ω, Resistor_SMD:R_0805_2012Metric_Pad1.20x1.40mm_HandSolder, symbol Device:R
- renumbered C19 to C16, C20 to C17, C22 to C18, C23 to C19, C24 to C20, C25 to C21, C26 to C22, C27 to C23, C28 to C24, C29 to C25, C30 to C26, C31 to C27, C32 to C28, C33 to C29, C34 to C30, C35 to C32, D6 to D4, D7 to D5, D8 to D6, R22 to R13, R23 to R14, R25 to R16, R26 to R17, R27 to R18, R28 to R19, U5 to U4
Connections:
- net +STM_3V3: now also R15.1
- net ADC1_IN6: now also C31.1
- net GND: now also C31.2
- net I2C1_SCL: now also R15.2
- net STM_LED renamed STM_LED_0
- net STM_LED_0: no longer D6.2 (A), R18.2
- new net STM_LED_1: D6.2 (A), R18.2
