File: hardware/kicad/STM32.kicad_sch (KiCad schematic)
At the start: 35 parts, among them J2 01x06_Pin, U4 STM32F411CEUx, Y1 YSX321SL, Y2 YST310S

Commit message: finished pcb
Parts:
- J3: renamed from J2; footprint Connector_PinHeader_2.54mm:PinHeader_1x06_P2.54mm_Vertical -> Connector_PinHeader_2.54mm:PinHeader_1x06_P2.54mm_Horizontal

Commit message: Final hardware cleanup push (hopefully)
Other:
- note added: "ADC FILTER CAPACITOR"
- note added: "ANALOG VDDA FILTERING"
- note added: "DECOUPLING CAPACITORS"
- note added: "INTER LDO CAPACITOR"
- note added: "STM32F411CEU6"
- note removed: "ANALOG FILTERING"
- note removed: "DECOUPLING CAPS"
- company: (none) -> Done By :- Arudhran
- title: (none) -> Cryptographic Tactical Node
- moved on the sheet: C16, C18, C21, C24, C27, C29, C30, C31, Y1, Y2
