File: hardware/kicad/GPS.kicad_sch (KiCad schematic)
At the start: 0 parts

Commit message: GPS and LoRA completed
Parts:
- added C44: 10μF, symbol Device:C
- added C45: 100nF, symbol Device:C
- added U7: NEO-M8N, NEO_M8N:NEO_M8N, symbol NEO_M8N:NEO_M8N
Connections:
- net GPS_RX: now also U7.2 (RX)
- net GPS_TX: now also U7.3 (TX)
- new net +5V: C44.1, C45.1, U7.1 (VCC)
- new net GND: C44.2, C45.2, U7.4 (GND)
Other:
- note added: "DECOUPLING CAPS"
- note added: "NEO-M8N GPS"
