File: hardware/kicad/GPS.kicad_sch (KiCad schematic)
At the start: 3 parts, among them U5 NEO-M8N

Commit message: finished pcb
Parts:
- added J4: Conn_01x02_Pin, Connector_PinHeader_2.54mm:PinHeader_1x02_P2.54mm_Vertical, symbol Connector:Conn_01x02_Pin
Connections:
- net GPS_RX: now also J4.2 (Pin_2)
- net GPS_TX: now also J4.1 (Pin_1)
Changed lines of the file:
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@@
+		)
+	)
+	(wire
+		(pts
+			(xy 81.28 39.37) (xy 74.93 39.37)
+		)
+		(stroke
+			(width 0)
+			(type default)
 		)
 	)
@@
 	(wire
 		(pts
+			(xy 81.28 41.91) (xy 74.93 41.91)
+		)
+		(stroke
+			(width 0)
+			(type default)
+		)
+	)
+	(wire
+		(pts
 			(xy 64.77 73.66) (xy 64.77 76.2)
 		)
@@
 			(width 0)
 			(type default)
+		)
+	)
+	(hierarchical_label "GPS_TX"
+		(shape output)
+		(at 81.28 39.37 0)
+		(effects
+			(font
+				(size 1.27 1.27)
+			)
+			(justify left)
+		)
+	)
+	(hierarchical_label "GPS_RX"
+		(shape input)
+		(at 81.28 41.91 0)
+		(effects
+			(font
+				(size 1.27 1.27)
+			)
+			(justify left)
 		)
 	)
@@
 		(dnp no)
 		(fields_autoplaced yes)
-		(property "Reference" "#PWR071"
+		(property "Reference" "#PWR072"
 			(at 69.85 85.09 0)
 			(hide yes)
@@
 			(project "crypto_node"
 				(path "/6c72b0cb-17b9-42a6-811c-297d0c354af3/e995d37b-7e81-489c-a8c7-4473f579a36c"
-					(reference "#PWR071")
+					(reference "#PWR072")
 					(unit 1)
 				)
@@
 		(in_pos_files yes)
 		(dnp no)
-		(property "Reference" "#PWR070"
+		(property "Reference" "#PWR071"
 			(at 69.85 64.77 0)
 			(hide yes)
@@
 			(project "crypto_node"
 				(path "/6c72b0cb-17b9-42a6-811c-297d0c354af3/e995d37b-7e81-489c-a8c7-4473f579a36c"
-					(reference "#PWR070")
+					(reference "#PWR071")
 					(unit 1)
 				)
@@
 		(dnp no)
 		(fields_autoplaced yes)
-		(property "Reference" "#PWR073"
+		(property "Reference" "#PWR074"
 			(at 130.81 59.69 0)
 			(hide yes)
@@
 			(project "crypto_node"
 				(path "/6c72b0cb-17b9-42a6-811c-297d0c354af3/e995d37b-7e81-489c-a8c7-4473f579a36c"
-					(reference "#PWR073")
+					(reference "#PWR074")
 					(unit 1)
 				)
@@
 		(in_pos_files yes)
 		(dnp no)
-		(property "Reference" "#PWR072"
+		(property "Reference" "#PWR073"
 			(at 102.87 44.45 0)
 			(hide yes)
@@
 			(project "crypto_node"
 				(path "/6c72b0cb-17b9-42a6-811c-297d0c354af3/e995d37b-7e81-489c-a8c7-4473f579a36c"
-					(reference "#PWR072")
+					(reference "#PWR073")
 					(unit 1)
 				)
+			)
+		)
+	)
+	(symbol
+		(lib_id "Connector:Conn_01x02_Pin")
+		(at 69.85 39.37 0)
+		(unit 1)
+		(body_style 1)
+		(exclude_from_sim no)
+		(in_bom yes)
+		(on_board yes)
+		(in_pos_files yes)
+		(dnp no)
+		(fields_autoplaced yes)
+		(property "Reference" "J4"
+			(at 70.485 34.29 0)
+			(show_name no)
+			(do_not_autoplace no)
+			(effects
+				(font
+					(size 1.27 1.27)
+				)
+			)
+		)
+		(property "Value" "Conn_01x02_Pin"
+			(at 70.485 36.83 0)
+			(show_name no)
+			(do_not_autoplace no)
+			(effects
+				(font
+					(size 1.27 1.27)
+				)
+			)
+		)
+		(property "Footprint" "Connector_PinHeader_2.54mm:PinHeader_1x02_P2.54mm_Vertical"
+			(at 69.85 39.37 0)
+			(hide yes)
+			(show_name no)
+			(do_not_autoplace no)
+			(effects
+				(font
+					(size 1.27 1.27)
+				)
+			)
+		)
+		(property "Datasheet" ""
+			(at 69.85 39.37 0)
+			(hide yes)
+			(show_name no)
+			(do_not_autoplace no)
+			(effects
+				(font
+					(size 1.27 1.27)
+				)
+			)
+		)
+		(property "Description" "Generic connector, single row, 01x02, script generated"
+			(at 69.85 39.37 0)
+			(hide yes)
+			(show_name no)
+			(do_not_autoplace no)
+			(effects
+				(font
+					(size 1.27 1.27)
+				)
+			)
+		)
+		(pin "1"
+		)
+		(pin "2"
+		)
+		(instances
+			(project "crypto_node"
+				(path "/6c72b0cb-17b9-42a6-811c-297d0c354af3/e995d37b-7e81-489c-a8c7-4473f579a36c"
+					(reference "J4")
+					(unit 1)
+				)

Commit message: Final hardware cleanup push (hopefully)
Other:
- note added: "DEBUGGING"
- company: (none) -> Done By :- Arudhran
- title: (none) -> Cryptographic Tactical Node
- moved on the sheet: J4
Changed lines of the file:
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@@
 	(generator_version "10.0")
 	(paper "A5")
+	(title_block
+		(title "Cryptographic Tactical Node")
+		(date "06-10-2020")
+		(company "Done By :- Arudhran")
+	)
 	(rectangle
 		(start 57.15 22.86)
@@
 	(text "NEO-M8N GPS"
 		(exclude_from_sim no)
-		(at 58.42 25.4 0)
+		(at 58.42 26.67 0)
 		(effects
 			(font
-				(face "JetBrainsMono NF")
-				(size 3 3)
+				(size 2.032 2.032)
+				(thickness 0.6)
 				(bold yes)
+				(italic yes)
 				(color 0 255 0 1)
 			)
-			(justify left top)
+			(justify left)
+		)
+	)
+	(text "DEBUGGING"
+		(exclude_from_sim no)
+		(at 58.42 54.61 0)
+		(effects
+			(font
+				(size 1.016 1.016)
+				(thickness 0.127)
+				(color 0 255 255 1)
+			)
+			(justify left)
 		)
 	)
@@
 		(color 0 0 0 0)
 	)
+	(polyline
+		(pts
+			(xy 57.15 35.56) (xy 83.82 35.56)
+		)
+		(stroke
+			(width 0)
+			(type dash_dot)
+		)
+	)
 	(wire
 		(pts
@@
 		(stroke
 			(width 0)
-			(type solid)
+			(type dash_dot)
 		)
 	)
@@
 	(polyline
 		(pts
+			(xy 57.15 52.07) (xy 83.82 52.07)
+		)
+		(stroke
+			(width 0)
+			(type dash_dot)
+		)
+	)
+	(polyline
+		(pts
 			(xy 57.15 55.88) (xy 83.82 55.88)
 		)
 		(stroke
 			(width 0)
-			(type default)
-		)
-	)
-	(wire
-		(pts
-			(xy 81.28 39.37) (xy 74.93 39.37)
+			(type dash_dot)
+		)
+	)
+	(wire
+		(pts
+			(xy 72.39 45.72) (xy 66.04 45.72)
 		)
 		(stroke
@@
 		)
 	)
+	(polyline
+		(pts
+			(xy 83.82 35.56) (xy 83.82 55.88)
+		)
+		(stroke
+			(width 0)
+			(type dash_dot)
+		)
+	)
 	(wire
 		(pts
@@
 		(stroke
 			(width 0)
-			(type default)
+			(type dash_dot)
 		)
 	)
@@
 		(stroke
 			(width 0)
-			(type default)
-		)
-	)
-	(wire
-		(pts
-			(xy 81.28 41.91) (xy 74.93 41.91)
+			(type dash_dot)
+		)
+	)
+	(wire
+		(pts
+			(xy 72.39 48.26) (xy 66.04 48.26)
 		)
 		(stroke
@@
 	(hierarchical_label "GPS_TX"
 		(shape output)
-		(at 81.28 39.37 0)
+		(at 72.39 45.72 0)
 		(effects
 			(font
@@
 	(hierarchical_label "GPS_RX"
 		(shape input)
-		(at 81.28 41.91 0)
+		(at 72.39 48.26 0)
 		(effects
 			(font
@@
 			)
 		)
+		(pin "3"
+		)
+		(pin "4"
+		)
 		(pin "1"
-		)
-		(pin "4"
-		)
-		(pin "3"
 		)
 		(pin "2"
@@
 	(symbol
 		(lib_id "Connector:Conn_01x02_Pin")
-		(at 69.85 39.37 0)
+		(at 60.96 45.72 0)
 		(unit 1)
 		(body_style 1)
@@
 		(in_pos_files yes)
 		(dnp no)
-		(fields_autoplaced yes)
 		(property "Reference" "J4"
-			(at 70.485 34.29 0)
+			(at 68.58 39.37 0)
 			(show_name no)
 			(do_not_autoplace no)
@@
 		)
 		(property "Value" "Conn_01x02_Pin"
-			(at 70.485 36.83 0)
+			(at 68.58 41.91 0)
 			(show_name no)
 			(do_not_autoplace no)
@@
 		)
 		(property "Footprint" "Connector_PinHeader_2.54mm:PinHeader_1x02_P2.54mm_Vertical"
-			(at 69.85 39.37 0)
+			(at 60.96 45.72 0)
 			(hide yes)
 			(show_name no)
@@
 		)
 		(property "Datasheet" ""
-			(at 69.85 39.37 0)
+			(at 60.96 45.72 0)
 			(hide yes)
 			(show_name no)
@@
 		)
 		(property "Description" "Generic connector, single row, 01x02, script generated"
-			(at 69.85 39.37 0)
-			(hide yes)
-			(show_name no)
+			(at 60.96 45.72 0)
+			(hide yes)
+			(show_name no)
