File: hardware/kicad/LoRA.kicad_sch (KiCad schematic)
At the start: 5 parts, among them U7 EBYTE_900T20D

Commit message: finished pcb
Parts:
- added J6: Conn_01x02_Pin, Connector_PinHeader_2.54mm:PinHeader_1x02_P2.54mm_Vertical, symbol Connector:Conn_01x02_Pin
Connections:
- net LORA_RX: now also J6.2 (Pin_2)
- net LORA_TX: now also J6.1 (Pin_1)
Changed lines of the file:
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@@
+	(wire
+		(pts
+			(xy 134.62 87.63) (xy 142.24 87.63)
+		)
+		(stroke
+			(width 0)
+			(type default)
+		)
+	)
 	(wire
 		(pts
@@
 	(wire
 		(pts
+			(xy 134.62 85.09) (xy 142.24 85.09)
+		)
+		(stroke
+			(width 0)
+			(type default)
+		)
+	)
+	(wire
+		(pts
 			(xy 137.16 62.23) (xy 137.16 64.77)
 		)
@@
 			(width 0)
 			(type default)
+		)
+	)
+	(hierarchical_label "LORA_RX"
+		(shape input)
+		(at 142.24 87.63 0)
+		(effects
+			(font
+				(size 1.27 1.27)
+			)
+			(justify left)
+		)
+	)
+	(hierarchical_label "LORA_TX"
+		(shape output)
+		(at 142.24 85.09 0)
+		(effects
+			(font
+				(size 1.27 1.27)
+			)
+			(justify left)
 		)
 	)
@@
 		(dnp no)
 		(fields_autoplaced yes)
-		(property "Reference" "#PWR083"
+		(property "Reference" "#PWR084"
 			(at 142.24 73.66 0)
 			(hide yes)
@@
 			(project "crypto_node"
 				(path "/6c72b0cb-17b9-42a6-811c-297d0c354af3/a6d9426e-b53a-46eb-ac04-bfb7b6f1fcf7"
-					(reference "#PWR083")
+					(reference "#PWR084")
 					(unit 1)
 				)
@@
 		(dnp no)
 		(fields_autoplaced yes)
-		(property "Reference" "#PWR079"
+		(property "Reference" "#PWR080"
 			(at 64.77 92.71 0)
 			(hide yes)
@@
 			(project "crypto_node"
 				(path "/6c72b0cb-17b9-42a6-811c-297d0c354af3/a6d9426e-b53a-46eb-ac04-bfb7b6f1fcf7"
-					(reference "#PWR079")
+					(reference "#PWR080")
 					(unit 1)
 				)
@@
 		(dnp no)
 		(fields_autoplaced yes)
-		(property "Reference" "#PWR081"
+		(property "Reference" "#PWR082"
 			(at 115.57 92.71 0)
 			(hide yes)
@@
 			(project "crypto_node"
 				(path "/6c72b0cb-17b9-42a6-811c-297d0c354af3/a6d9426e-b53a-46eb-ac04-bfb7b6f1fcf7"
-					(reference "#PWR081")
+					(reference "#PWR082")
+					(unit 1)
+				)
+			)
+		)
+	)
+	(symbol
+		(lib_id "Connector:Conn_01x02_Pin")
+		(at 129.54 85.09 0)
+		(unit 1)
+		(body_style 1)
+		(exclude_from_sim no)
+		(in_bom yes)
+		(on_board yes)
+		(in_pos_files yes)
+		(dnp no)
+		(fields_autoplaced yes)
+		(property "Reference" "J6"
+			(at 130.175 80.01 0)
+			(show_name no)
+			(do_not_autoplace no)
+			(effects
+				(font
+					(size 1.27 1.27)
+				)
+			)
+		)
+		(property "Value" "Conn_01x02_Pin"
+			(at 130.175 82.55 0)
+			(show_name no)
+			(do_not_autoplace no)
+			(effects
+				(font
+					(size 1.27 1.27)
+				)
+			)
+		)
+		(property "Footprint" "Connector_PinHeader_2.54mm:PinHeader_1x02_P2.54mm_Vertical"
+			(at 129.54 85.09 0)
+			(hide yes)
+			(show_name no)
+			(do_not_autoplace no)
+			(effects
+				(font
+					(size 1.27 1.27)
+				)
+			)
+		)
+		(property "Datasheet" ""
+			(at 129.54 85.09 0)
+			(hide yes)
+			(show_name no)
+			(do_not_autoplace no)
+			(effects
+				(font
+					(size 1.27 1.27)
+				)
+			)
+		)
+		(property "Description" "Generic connector, single row, 01x02, script generated"
+			(at 129.54 85.09 0)
+			(hide yes)
+			(show_name no)
+			(do_not_autoplace no)
+			(effects
+				(font
+					(size 1.27 1.27)
+				)
+			)
+		)
+		(pin "1"
+		)
+		(pin "2"
+		)
+		(instances
+			(project "crypto_node"
+				(path "/6c72b0cb-17b9-42a6-811c-297d0c354af3/a6d9426e-b53a-46eb-ac04-bfb7b6f1fcf7"
+					(reference "J6")
 					(unit 1)
 				)
@@
 		(dnp no)
 		(fields_autoplaced yes)
-		(property "Reference" "#PWR080"
+		(property "Reference" "#PWR081"
 			(at 115.57 49.53 0)
 			(hide yes)
@@
 			(project "crypto_node"
 				(path "/6c72b0cb-17b9-42a6-811c-297d0c354af3/a6d9426e-b53a-46eb-ac04-bfb7b6f1fcf7"
-					(reference "#PWR080")
+					(reference "#PWR081")
 					(unit 1)
 				)
@@
 		(in_pos_files yes)
 		(dnp no)
-		(property "Reference" "#PWR082"
+		(property "Reference" "#PWR083"
 			(at 142.24 53.34 0)
 			(hide yes)
@@
 			(project "crypto_node"
 				(path "/6c72b0cb-17b9-42a6-811c-297d0c354af3/a6d9426e-b53a-46eb-ac04-bfb7b6f1fcf7"
-					(reference "#PWR082")
+					(reference "#PWR083")
 					(unit 1)
 				)

Commit message: Final hardware cleanup push (hopefully)
Other:
- note added: "DEBUGGING"
- company: (none) -> Done By :- Arudhran
- title: (none) -> Cryptographic Tactical Node
- moved on the sheet: J6
Changed lines of the file:
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@@
 	(generator_version "10.0")
 	(paper "A5")
+	(title_block
+		(title "Cryptographic Tactical Node")
+		(date "06-10-2020")
+		(company "Done By :- Arudhran")
+	)
 	(rectangle
 		(start 57.15 31.75)
@@
 	(text "EBYTE 900T20D LoRA"
 		(exclude_from_sim no)
-		(at 58.42 34.29 0)
+		(at 58.42 35.56 0)
 		(effects
 			(font
-				(face "JetBrainsMono NF")
-				(size 3 3)
+				(size 2.032 2.032)
 				(bold yes)
+				(italic yes)
 				(color 0 255 0 1)
 			)
-			(justify left top)
+			(justify left)
 		)
 	)
@@
 		)
 	)
+	(text "DEBUGGING"
+		(exclude_from_sim no)
+		(at 130.81 92.71 0)
+		(effects
+			(font
+				(size 1.016 1.016)
+				(thickness 0.127)
+				(color 0 255 255 1)
+			)
+			(justify left)
+		)
+	)
 	(junction
 		(at 81.28 68.58)
@@
 		)
 	)
-	(wire
-		(pts
-			(xy 134.62 87.63) (xy 142.24 87.63)
+	(polyline
+		(pts
+			(xy 129.54 76.2) (xy 129.54 93.98)
+		)
+		(stroke
+			(width 0)
+			(type dash_dot)
+		)
+	)
+	(wire
+		(pts
+			(xy 137.16 86.36) (xy 144.78 86.36)
 		)
 		(stroke
@@
 		)
 	)
+	(polyline
+		(pts
+			(xy 129.54 90.17) (xy 154.94 90.17)
+		)
+		(stroke
+			(width 0)
+			(type dash_dot)
+		)
+	)
 	(wire
 		(pts
@@
 		(stroke
 			(width 0)
-			(type default)
-		)
-	)
-	(wire
-		(pts
-			(xy 134.62 85.09) (xy 142.24 85.09)
+			(type dash_dot)
+		)
+	)
+	(wire
+		(pts
+			(xy 137.16 83.82) (xy 144.78 83.82)
 		)
 		(stroke
@@
 		(stroke
 			(width 0)
-			(type default)
+			(type dash_dot)
 		)
 	)
@@
 		(stroke
 			(width 0)
-			(type default)
+			(type dash_dot)
 		)
 	)
@@
 		(stroke
 			(width 0)
-			(type default)
+			(type dash_dot)
 		)
 	)
@@
 	(hierarchical_label "LORA_RX"
 		(shape input)
-		(at 142.24 87.63 0)
+		(at 144.78 86.36 0)
 		(effects
 			(font
@@
 	(hierarchical_label "LORA_TX"
 		(shape output)
-		(at 142.24 85.09 0)
+		(at 144.78 83.82 0)
 		(effects
 			(font
@@
 	(symbol
 		(lib_id "Connector:Conn_01x02_Pin")
-		(at 129.54 85.09 0)
+		(at 132.08 83.82 0)
 		(unit 1)
 		(body_style 1)
@@
 		(in_pos_files yes)
 		(dnp no)
-		(fields_autoplaced yes)
 		(property "Reference" "J6"
-			(at 130.175 80.01 0)
+			(at 132.715 78.74 0)
 			(show_name no)
 			(do_not_autoplace no)
@@
 		)
 		(property "Value" "Conn_01x02_Pin"
-			(at 130.175 82.55 0)
+			(at 139.7 81.28 0)
 			(show_name no)
 			(do_not_autoplace no)
@@
 		)
 		(property "Footprint" "Connector_PinHeader_2.54mm:PinHeader_1x02_P2.54mm_Vertical"
-			(at 129.54 85.09 0)
+			(at 132.08 83.82 0)
 			(hide yes)
 			(show_name no)
@@
 		)
 		(property "Datasheet" ""
-			(at 129.54 85.09 0)
+			(at 132.08 83.82 0)
 			(hide yes)
 			(show_name no)
@@
 		)
 		(property "Description" "Generic connector, single row, 01x02, script generated"
-			(at 129.54 85.09 0)
-			(hide yes)
-			(show_name no)
+			(at 132.08 83.82 0)
+			(hide yes)
+			(show_name no)
