File: hardware/kicad/Crypt.kicad_sch (KiCad schematic)
At the start: 3 parts, among them U9 SE050

Commit message: schematics refinement
Parts:
- C38: renamed from C48; footprint (none) -> Capacitor_SMD:C_1206_3216Metric_Pad1.33x1.80mm_HandSolder
- C39: renamed from C49; footprint (none) -> Capacitor_SMD:C_0603_1608Metric_Pad1.08x0.95mm_HandSolder
- U7: renamed from U9; footprint (none) -> HX2QFN20:HX2QFN20
Changed lines of the file:
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@@
 		(in_pos_files yes)
 		(dnp no)
-		(property "Reference" "#PWR097"
+		(property "Reference" "#PWR087"
 			(at 104.14 57.15 0)
 			(hide yes)
@@
 			(project "crypto_node"
 				(path "/6c72b0cb-17b9-42a6-811c-297d0c354af3/b388d7dd-e85d-4888-b4a4-ed6170d89183"
-					(reference "#PWR097")
+					(reference "#PWR087")
 					(unit 1)
 				)
@@
 		(in_pos_files yes)
 		(dnp no)
-		(property "Reference" "C49"
+		(property "Reference" "C39"
 			(at 138.43 67.31 0)
 			(show_name no)
@@
 			)
 		)
-		(property "Footprint" ""
+		(property "Footprint" "Capacitor_SMD:C_0603_1608Metric_Pad1.08x0.95mm_HandSolder"
 			(at 138.1252 73.66 0)
 			(hide yes)
@@
 			(project "crypto_node"
 				(path "/6c72b0cb-17b9-42a6-811c-297d0c354af3/b388d7dd-e85d-4888-b4a4-ed6170d89183"
-					(reference "C49")
+					(reference "C39")
 					(unit 1)
 				)
@@
 		(in_pos_files yes)
 		(dnp no)
-		(property "Reference" "#PWR0100"
+		(property "Reference" "#PWR088"
 			(at 132.08 64.77 0)
 			(hide yes)
@@
 			(project "crypto_node"
 				(path "/6c72b0cb-17b9-42a6-811c-297d0c354af3/b388d7dd-e85d-4888-b4a4-ed6170d89183"
-					(reference "#PWR0100")
+					(reference "#PWR088")
 					(unit 1)
 				)
@@
 		(dnp no)
 		(fields_autoplaced yes)
-		(property "Reference" "#PWR096"
+		(property "Reference" "#PWR086"
 			(at 86.36 93.98 0)
 			(hide yes)
@@
 			(project "crypto_node"
 				(path "/6c72b0cb-17b9-42a6-811c-297d0c354af3/b388d7dd-e85d-4888-b4a4-ed6170d89183"
-					(reference "#PWR096")
+					(reference "#PWR086")
 					(unit 1)
 				)
@@
 		(in_pos_files yes)
 		(dnp no)
-		(property "Reference" "C48"
+		(property "Reference" "C38"
 			(at 128.27 67.31 0)
 			(show_name no)
@@
 			)
 		)
-		(property "Footprint" ""
+		(property "Footprint" "Capacitor_SMD:C_1206_3216Metric_Pad1.33x1.80mm_HandSolder"
 			(at 127.9652 73.66 0)
 			(hide yes)
@@
 			(project "crypto_node"
 				(path "/6c72b0cb-17b9-42a6-811c-297d0c354af3/b388d7dd-e85d-4888-b4a4-ed6170d89183"
-					(reference "C48")
+					(reference "C38")
 					(unit 1)
 				)
@@
 		(dnp no)
 		(fields_autoplaced yes)
-		(property "Reference" "#PWR098"
+		(property "Reference" "#PWR085"
 			(at 66.04 93.98 0)
 			(hide yes)
@@
 			(project "crypto_node"
 				(path "/6c72b0cb-17b9-42a6-811c-297d0c354af3/b388d7dd-e85d-4888-b4a4-ed6170d89183"
-					(reference "#PWR098")
+					(reference "#PWR085")
 					(unit 1)
 				)
@@
 		(dnp no)
 		(fields_autoplaced yes)
-		(property "Reference" "#PWR0101"
+		(property "Reference" "#PWR089"
 			(at 132.08 85.09 0)
 			(hide yes)
@@
 			(project "crypto_node"
 				(path "/6c72b0cb-17b9-42a6-811c-297d0c354af3/b388d7dd-e85d-4888-b4a4-ed6170d89183"
-					(reference "#PWR0101")
+					(reference "#PWR089")
 					(unit 1)
 				)
@@
 		(dnp no)
 		(fields_autoplaced yes)
-		(property "Reference" "U9"
+		(property "Reference" "U7"
 			(at 85.09 50.8 0)
 			(show_name no)
@@
 			)
 		)
-		(property "Footprint" ""
+		(property "Footprint" "HX2QFN20:HX2QFN20"
 			(at 85.09 68.58 0)
 			(hide yes)
@@
 			(project "crypto_node"
 				(path "/6c72b0cb-17b9-42a6-811c-297d0c354af3/b388d7dd-e85d-4888-b4a4-ed6170d89183"
-					(reference "U9")
-					(unit 1)
-				)
+					(reference "U7")
+					(unit 1)
+				)

Commit message: started PCB and changed power system
Parts:
- renumbered C38 to C35, C39 to C36, U7 to U6
Changed lines of the file:
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@@
 		(in_pos_files yes)
 		(dnp no)
-		(property "Reference" "#PWR087"
+		(property "Reference" "#PWR077"
 			(at 104.14 57.15 0)
 			(hide yes)
@@
 			(project "crypto_node"
 				(path "/6c72b0cb-17b9-42a6-811c-297d0c354af3/b388d7dd-e85d-4888-b4a4-ed6170d89183"
-					(reference "#PWR087")
+					(reference "#PWR077")
 					(unit 1)
 				)
@@
 		(in_pos_files yes)
 		(dnp no)
-		(property "Reference" "C39"
+		(property "Reference" "C36"
 			(at 138.43 67.31 0)
 			(show_name no)
@@
 			(project "crypto_node"
 				(path "/6c72b0cb-17b9-42a6-811c-297d0c354af3/b388d7dd-e85d-4888-b4a4-ed6170d89183"
-					(reference "C39")
+					(reference "C36")
 					(unit 1)
 				)
@@
 		(in_pos_files yes)
 		(dnp no)
-		(property "Reference" "#PWR088"
+		(property "Reference" "#PWR078"
 			(at 132.08 64.77 0)
 			(hide yes)
@@
 			(project "crypto_node"
 				(path "/6c72b0cb-17b9-42a6-811c-297d0c354af3/b388d7dd-e85d-4888-b4a4-ed6170d89183"
-					(reference "#PWR088")
+					(reference "#PWR078")
 					(unit 1)
 				)
@@
 		(dnp no)
 		(fields_autoplaced yes)
-		(property "Reference" "#PWR086"
+		(property "Reference" "#PWR076"
 			(at 86.36 93.98 0)
 			(hide yes)
@@
 			(project "crypto_node"
 				(path "/6c72b0cb-17b9-42a6-811c-297d0c354af3/b388d7dd-e85d-4888-b4a4-ed6170d89183"
-					(reference "#PWR086")
+					(reference "#PWR076")
 					(unit 1)
 				)
@@
 		(in_pos_files yes)
 		(dnp no)
-		(property "Reference" "C38"
+		(property "Reference" "C35"
 			(at 128.27 67.31 0)
 			(show_name no)
@@
 			(project "crypto_node"
 				(path "/6c72b0cb-17b9-42a6-811c-297d0c354af3/b388d7dd-e85d-4888-b4a4-ed6170d89183"
-					(reference "C38")
+					(reference "C35")
 					(unit 1)
 				)
@@
 		(dnp no)
 		(fields_autoplaced yes)
-		(property "Reference" "#PWR085"
+		(property "Reference" "#PWR075"
 			(at 66.04 93.98 0)
 			(hide yes)
@@
 			(project "crypto_node"
 				(path "/6c72b0cb-17b9-42a6-811c-297d0c354af3/b388d7dd-e85d-4888-b4a4-ed6170d89183"
-					(reference "#PWR085")
+					(reference "#PWR075")
 					(unit 1)
 				)
@@
 		(dnp no)
 		(fields_autoplaced yes)
-		(property "Reference" "#PWR089"
+		(property "Reference" "#PWR079"
 			(at 132.08 85.09 0)
 			(hide yes)
@@
 			(project "crypto_node"
 				(path "/6c72b0cb-17b9-42a6-811c-297d0c354af3/b388d7dd-e85d-4888-b4a4-ed6170d89183"
-					(reference "#PWR089")
+					(reference "#PWR079")
 					(unit 1)
 				)
@@
 		(dnp no)
 		(fields_autoplaced yes)
-		(property "Reference" "U7"
+		(property "Reference" "U6"
 			(at 85.09 50.8 0)
 			(show_name no)
@@
 			(project "crypto_node"
 				(path "/6c72b0cb-17b9-42a6-811c-297d0c354af3/b388d7dd-e85d-4888-b4a4-ed6170d89183"
-					(reference "U7")
-					(unit 1)
-				)
+					(reference "U6")
+					(unit 1)
+				)
