File: hardware/kicad/Crypt.kicad_sch (KiCad schematic)
At the start: 5 parts, among them U6 SE050

Commit message: finished pcb
Parts:
- added TP1, TP2, TP3: TestPoint, TestPoint:TestPoint_Pad_D1.5mm, symbol Connector:TestPoint
Connections:
- net CRYPT_SCL: now also TP1.1
- net CRYPT_SDA: now also TP2.1
- net GND: now also TP3.1
