File: hardware/kicad/Crypt.kicad_sch (KiCad schematic)
At the start: 8 parts, among them U6 SE050

Commit message: Final hardware cleanup push (hopefully)
Other:
- note added: "DEBUGGING"
- company: (none) -> Done By :- Arudhran
- title: (none) -> Cryptographic Tactical Node
- moved on the sheet: C35, C36, R18, R19, TP1, TP2, TP3
