File: hardware/kicad/crypto_node.kicad_pcb (KiCad board)
At the start: 2 copper layers, 107 parts, among them J1 USB_C_Receptacle_USB2.0_16P, J2 01x06_Pin, Q1 FDN304PZ, SW1 SW_SPDT_321, U1 TPS61023DRLR, U2 MCP73871-2CC, U3 TLV74333PDBVR, U4 TLV74333PDBVR, U5 STM32F411CEUx, U6 NEO-M8N, U7 SE050, U8 EBYTE_900T20D, Y1 YSX321SL, Y2 YST310S

Commit message: started PCB and changed power system
Parts:
- removed C18, C27, C41, C42: 100nF, Capacitor_SMD:C_0603_1608Metric_Pad1.08x0.95mm_HandSolder
- removed C40: 10μF, Capacitor_SMD:C_1206_3216Metric_Pad1.33x1.80mm_HandSolder
- removed D7, D8: white, LED_SMD:LED_0805_2012Metric_Pad1.15x1.40mm_HandSolder
- removed NT1, NT2, NT3, NT4: NetTie_2, NetTie:NetTie-2_SMD_Pad0.5mm
- removed R23: 10KΩ, Resistor_SMD:R_0805_2012Metric_Pad1.20x1.40mm_HandSolder
- removed R24: 4K7Ω, Resistor_SMD:R_0805_2012Metric_Pad1.20x1.40mm_HandSolder
- removed R25: 2K2Ω, Resistor_SMD:R_0805_2012Metric_Pad1.20x1.40mm_HandSolder
- removed R26, R27: 470Ω, Resistor_SMD:R_0805_2012Metric_Pad1.20x1.40mm_HandSolder
- removed R28, R29, R30, R31: 33KΩ, Resistor_SMD:R_0805_2012Metric_Pad1.20x1.40mm_HandSolder
- removed U8: EBYTE_900T20D, EBYTE_900T20D:EBYTE_900T20D
- added BT2: 18650 Li-ion, Battery:BatteryHolder_Keystone_1042_1x18650, B.Cu at (166.9, 71.6)
- added C22: 100nF, Capacitor_SMD:C_0603_1608Metric_Pad1.08x0.95mm_HandSolder, F.Cu at (175.4, 84.1)
- added C31: 100nF, Capacitor_SMD:C_0603_1608Metric_Pad1.08x0.95mm_HandSolder, F.Cu at (174.3, 69.4)
- added F1: OZCF0185FF2C, Fuse:Fuse_2920_7451Metric_Pad2.10x5.45mm_HandSolder, B.Cu at (199.1, 114.8)
- added H1: Mount_Hole, MountingHole:MountingHole_3.2mm_M3_Pad_Via, F.Cu at (88.4, 62.7)
- added H2: Mount_Hole, MountingHole:MountingHole_3.2mm_M3_Pad_Via, F.Cu at (88.4, 120.3)
- added H3: Mount_Hole, MountingHole:MountingHole_3.2mm_M3_Pad_Via, F.Cu at (210.0, 62.7)
- added H4: Mount_Hole, MountingHole:MountingHole_3.2mm_M3_Pad_Via, F.Cu at (210.0, 120.3)
- BT1: value 103450 Li-PO -> 18650 Li-ion; footprint Connector_JST:JST_PH_B2B-PH-K_1x02_P2.00mm_Vertical -> Battery:BatteryHolder_Keystone_1042_1x18650; moved to B.Cu
- C1, C11, C12, C17, C32, C37: value 100nF -> 10μF; footprint Capacitor_SMD:C_0603_1608Metric_Pad1.08x0.95mm_HandSolder -> Capacitor_SMD:C_1206_3216Metric_Pad1.33x1.80mm_HandSolder
- C14, C15, C20, C36, C38, C8, C9: value 10μF -> 100nF; footprint Capacitor_SMD:C_1206_3216Metric_Pad1.33x1.80mm_HandSolder -> Capacitor_SMD:C_0603_1608Metric_Pad1.08x0.95mm_HandSolder
- C16: value 10μF -> 33pF; footprint Capacitor_SMD:C_1206_3216Metric_Pad1.33x1.80mm_HandSolder -> Capacitor_SMD:C_0402_1005Metric_Pad0.74x0.62mm_HandSolder
- C19: value 33pF -> 100nF; footprint Capacitor_SMD:C_0402_1005Metric_Pad0.74x0.62mm_HandSolder -> Capacitor_SMD:C_0603_1608Metric_Pad1.08x0.95mm_HandSolder
- C21: value 100nF -> 22pF; footprint Capacitor_SMD:C_0603_1608Metric_Pad1.08x0.95mm_HandSolder -> Capacitor_SMD:C_0402_1005Metric_Pad0.74x0.62mm_HandSolder
- C24: value 100nF -> 18pF; footprint Capacitor_SMD:C_0603_1608Metric_Pad1.08x0.95mm_HandSolder -> Capacitor_SMD:C_0402_1005Metric_Pad0.74x0.62mm_HandSolder
- C25: value 22pF -> 100nF; footprint Capacitor_SMD:C_0402_1005Metric_Pad0.74x0.62mm_HandSolder -> Capacitor_SMD:C_0603_1608Metric_Pad1.08x0.95mm_HandSolder
- C28: value 18pF -> 100nF; footprint Capacitor_SMD:C_0402_1005Metric_Pad0.74x0.62mm_HandSolder -> Capacitor_SMD:C_0603_1608Metric_Pad1.08x0.95mm_HandSolder
- C29: value 100nF -> 11pF; footprint Capacitor_SMD:C_0603_1608Metric_Pad1.08x0.95mm_HandSolder -> Capacitor_SMD:C_0402_1005Metric_Pad0.74x0.62mm_HandSolder
- C30: value 100nF -> 4μ7F; footprint Capacitor_SMD:C_0603_1608Metric_Pad1.08x0.95mm_HandSolder -> Capacitor_SMD:C_0805_2012Metric_Pad1.18x1.45mm_HandSolder
- C33: value 11pF -> 10μF; footprint Capacitor_SMD:C_0402_1005Metric_Pad0.74x0.62mm_HandSolder -> Capacitor_SMD:C_1206_3216Metric_Pad1.33x1.80mm_HandSolder
- C34: value 4μ7F -> 100nF; footprint Capacitor_SMD:C_0805_2012Metric_Pad1.18x1.45mm_HandSolder -> Capacitor_SMD:C_0603_1608Metric_Pad1.08x0.95mm_HandSolder
- C5: value 22μF -> 100nF; footprint Capacitor_SMD:C_1210_3225Metric_Pad1.33x2.70mm_HandSolder -> Capacitor_SMD:C_0603_1608Metric_Pad1.08x0.95mm_HandSolder
- C7: value 100nF -> 22μF; footprint Capacitor_SMD:C_0603_1608Metric_Pad1.08x0.95mm_HandSolder -> Capacitor_SMD:C_1210_3225Metric_Pad1.33x2.70mm_HandSolder
- D2, Q1, R8: moved to B.Cu
- D3: value white -> SS24B-Slkor; footprint LED_SMD:LED_0805_2012Metric_Pad1.15x1.40mm_HandSolder -> Diode_SMD:D_SMA
- D4: value white -> WS2812B-2020; footprint LED_SMD:LED_0805_2012Metric_Pad1.15x1.40mm_HandSolder -> LED_SMD:LED_WS2812B-2020_PLCC4_2.0x2.0mm
- D6: value WS2812B-2020 -> white; footprint LED_SMD:LED_WS2812B-2020_PLCC4_2.0x2.0mm -> LED_SMD:LED_0805_2012Metric_Pad1.15x1.40mm_HandSolder
- L1: value SWPA5040S1R0NT -> SWPA5040S3R3NT 3μ3h
- R10: value 100KΩ -> 10KΩ
- R11: value 270KΩ -> 33KΩ
- R12: value 100KΩ -> 5K1Ω
- R13: value 3K3Ω -> 10KΩ
- R14: value 33KΩ -> 10KΩ
- R15: value 10KΩ -> 5K1Ω
- R16: value 470Ω -> 2K2Ω
- R22: value 10KΩ -> 33KΩ
- R5: value 1KΩ -> 5K1Ω
- R9: value 732KΩ -> 54K9Ω
- U1: value TPS61023DRLR -> TPS563201; footprint Package_TO_SOT_SMD:SOT-563 -> Package_TO_SOT_SMD:SOT-23-6
- U2: value MCP73871-2CC -> TLV74333PDBVR; footprint Package_DFN_QFN:QFN-20-1EP_4x4mm_P0.5mm_EP2.5x2.5mm_ThermalVias -> Package_TO_SOT_SMD:SOT-23-5_HandSoldering
- U4: value TLV74333PDBVR -> STM32F411CEUx; footprint Package_TO_SOT_SMD:SOT-23-5_HandSoldering -> Package_DFN_QFN:QFN-48-1EP_7x7mm_P0.5mm_EP5.6x5.6mm
- U5: value STM32F411CEUx -> NEO-M8N; footprint Package_DFN_QFN:QFN-48-1EP_7x7mm_P0.5mm_EP5.6x5.6mm -> NEO_M8N:NEO_M8N
- U6: value NEO-M8N -> SE050; footprint NEO_M8N:NEO_M8N -> HX2QFN20:HX2QFN20
- U7: value SE050 -> EBYTE_900T20D; footprint HX2QFN20:HX2QFN20 -> EBYTE_900T20D:EBYTE_900T20D
- moved Q1 446.3 mm to (209.9, 108.0), turned to 90 degrees
- moved R8 441.5 mm to (209.9, 112.9), turned to 90 degrees
- moved D2 435.4 mm to (205.4, 112.8), turned to -90 degrees
- moved D5 419.4 mm to (209.9, 81.9)
- moved R17 410.5 mm to (209.9, 79.4), turned to 180 degrees
- moved R18 410.0 mm to (209.9, 87.0), turned to 180 degrees
- moved BT1 402.5 mm to (166.9, 96.1), turned to 180 degrees
- moved D4 400.2 mm to (189.7, 76.9), turned to 0 degrees
- moved C3 394.2 mm to (152.0, 113.6), turned to 180 degrees
- moved J1 392.7 mm to (154.3, 119.9)
- moved R12 390.9 mm to (187.5, 111.8)
- moved R6 387.6 mm to (152.7, 119.9), turned to 90 degrees
- moved R11 386.5 mm to (183.1, 111.8)
- moved R7 386.3 mm to (155.9, 119.9), turned to 90 degrees
- moved R16 384.0 mm to (177.7, 87.7), turned to 180 degrees
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Connections:
- BT1 pad 2: GND -> Net-(BT1--)
- C10 pad 1: +MCP_OUT -> +5V
- C12 pad 1: +5V -> +STM_3V3
- C13 pad 1: +5V -> +CRYPT_3V3
- C14 pad 1: +5V -> +STM_3V3
- C15 pad 1: +STM_3V3 -> +CRYPT_3V3
- C16 pad 1: +CRYPT_3V3 -> RCC_OSC_OUT
- C19 pad 1: RCC_OSC_OUT -> BOOT0
- C21 pad 1: +STM_3V3 -> RCC_OSC_IN
- C23 pad 1: BOOT0 -> NRST
- C24 pad 1: +STM_3V3 -> RCC_OSC32_IN
- C25 pad 1: RCC_OSC_IN -> +STM_3V3
- C26 pad 1: +STM_3V3 -> +STM_3V3_A
- C28 pad 1: RCC_OSC32_IN -> +STM_3V3
- C29 pad 1: +STM_3V3 -> RCC_OSC32_OUT
- C30 pad 1: +STM_3V3_A -> /STM32/VCAP_1
- C33 pad 1: RCC_OSC32_OUT -> +5V
- C34 pad 1: /STM32/VCAP_1 -> +5V
- C35 pad 1: +STM_3V3 -> +CRYPT_3V3
- C36 pad 1: +5V -> +CRYPT_3V3
- C38 pad 1: +CRYPT_3V3 -> +5V
- C39 pad 1: +CRYPT_3V3 -> /STM32/PC13
- C5 pad 1: +5V -> /Power/VBST
- C5 pad 2: GND -> /Power/SW
- C8 pad 1: +VUSB -> +5V
- C9 pad 1: +BATT_PROC -> +5V
- D2 pad 1: +BATT_PROC -> Net-(D2-K)
- D3 pad 1: Net-(D3-K) -> +5V
- D4 pad 1: Net-(D4-K) -> unconnected-(D4-DOUT-Pad1)
- D4 pad 2: +VUSB -> GND
- D5 pad 1: Net-(D5-K) -> GND
- D5 pad 2: +VUSB -> /STM32/STM_LED_0
- D6 pad 1: unconnected-(D6-DOUT-Pad1) -> GND
- D6 pad 2: GND -> /STM32/STM_LED_1
- L1 pad 1: +VCOM -> /Power/SW
- L1 pad 2: /Power/TPS_SW -> +5V
- Q1 pad 2: +BATT_PROC -> Net-(D2-K)
- R10 pad 1: /Power/TPS_FB -> /Power/VFB
- R11 pad 1: +VUSB -> +VCOM
- R11 pad 2: /Power/VPCC -> /Power/BATTERY_VOLTAGE
- R12 pad 1: /Power/VPCC -> /Power/BATTERY_VOLTAGE
- R13 pad 1: PROG1 -> +STM_3V3
- R13 pad 2: GND -> NRST
- R14 pad 1: PROG3 -> BOOT0
- R15 pad 1: THERM -> +STM_3V3
- R15 pad 2: GND -> /Crypt/CRYPT_SCL
- R16 pad 1: /Power/~{PG} -> +STM_3V3
- R16 pad 2: Net-(D3-K) -> /Crypt/CRYPT_SDA
- R17 pad 1: /Power/~{LBO} -> STATUS_LED_0
- R17 pad 2: Net-(D4-K) -> /STM32/STM_LED_0
- R18 pad 1: /Power/STAT2 -> STATUS_LED_1
- R18 pad 2: Net-(D5-K) -> /STM32/STM_LED_1
- R19 pad 1: +VCOM -> BOOT1
- R19 pad 2: /Power/POWER_VOLTAGE -> GND
- R20 pad 1: /Power/POWER_VOLTAGE -> /LoRA/LORA_M0
- R21 pad 1: +VUSB -> /LoRA/LORA_M1
- R22 pad 2: NRST -> /STM32/PC13
- R5 pad 2: /Power/TPS_EN -> /Power/EN
- R9 pad 2: /Power/TPS_FB -> /Power/VFB
- SW1 pad 2: +MCP_OUT -> +BATT_PROC
- U1 pad 1: /Power/TPS_FB -> GND
- U1 pad 2: /Power/TPS_EN -> /Power/SW
- U1 pad 4: GND -> /Power/VFB
- U1 pad 5: /Power/TPS_SW -> /Power/EN
- U1 pad 6: +5V -> /Power/VBST
- U2 pad 1: +MCP_OUT -> +5V
- U2 pad 2: /Power/VPCC -> GND
- U2 pad 3: SEL -> +5V
- U2 pad 4: PROG2 -> unconnected-(U2-NC-Pad4)
- U2 pad 5: THERM -> +STM_3V3
- U3 pad 5: +STM_3V3 -> +CRYPT_3V3
- U4 pad 1: +5V -> +STM_3V3
- U4 pad 2: GND -> /STM32/PC13
- U4 pad 3: +5V -> RCC_OSC32_IN
- U4 pad 4: unconnected-(U4-NC-Pad4) -> RCC_OSC32_OUT
- U4 pad 5: +CRYPT_3V3 -> RCC_OSC_IN
- U5 pad 1: +STM_3V3 -> +5V
- U5 pad 2: /STM32/PC13 -> /GPS/GPS_RX
- U5 pad 3: RCC_OSC32_IN -> /GPS/GPS_TX
- U5 pad 4: RCC_OSC32_OUT -> GND
- U6 pad 1: +5V -> GND
- U6 pad 2: /GPS/GPS_RX -> unconnected-(U6-NC-Pad2)
- U6 pad 3: /GPS/GPS_TX -> unconnected-(U6-ISO7816_IO1-Pad3)
- U6 pad 4: GND -> unconnected-(U6-NC-Pad4)
- U7 pad 1: GND -> /LoRA/LORA_M0
- U7 pad 10: /Crypt/CRYPT_SCL -> unconnected-(U7-NC-Pad10)
- U7 pad 2: unconnected-(U7-NC-Pad2) -> /LoRA/LORA_M1
- U7 pad 3: unconnected-(U7-ISO7816_IO1-Pad3) -> /LoRA/LORA_RX
- U7 pad 4: unconnected-(U7-NC-Pad4) -> /LoRA/LORA_TX
- U7 pad 5: unconnected-(U7-NC-Pad5) -> /LoRA/AUX
- U7 pad 6: unconnected-(U7-NC-Pad6) -> +5V
- U7 pad 7: unconnected-(U7-NC-Pad7) -> GND
- U7 pad 9: /Crypt/CRYPT_SDA -> unconnected-(U7-NC-Pad9)
Other:
- board outline added: 129.4 x 65.4 mm

Commit message: completd PCB (at least that's what I believe)
Parts:
- removed the R15 at (173.6, 87.7)
- removed the R16 at (177.7, 87.7)
- added R18: 2K2Ω, Resistor_SMD:R_0805_2012Metric_Pad1.20x1.40mm_HandSolder, F.Cu at (163.6, 89.4)
- added R19: 5K1Ω, Resistor_SMD:R_0805_2012Metric_Pad1.20x1.40mm_HandSolder, F.Cu at (159.4, 89.4)
- moved S2 52.2 mm to (188.7, 100.5), turned to 180 degrees
- moved S1 48.0 mm to (188.7, 96.1), turned to 0 degrees
- moved R14 47.4 mm to (183.7, 100.5), turned to 90 degrees
- moved C19 45.4 mm to (181.4, 100.5), turned to 90 degrees
- moved R13 42.8 mm to (183.7, 96.1), turned to 90 degrees
- moved C23 40.5 mm to (181.4, 96.1), turned to -90 degrees
- moved C32 36.9 mm to (153.7, 65.9)
- moved D4 36.9 mm to (153.7, 69.0)
- moved C39 27.4 mm to (171.8, 90.2)
- moved JP4 27.4 mm to (181.2, 90.2)
- moved R22 27.4 mm to (176.3, 93.5)
- moved S3 27.4 mm to (176.3, 90.2)
- moved JP3 16.5 mm to (149.2, 69.3), turned to 90 degrees
- moved C25 14.6 mm to (152.5, 84.0), turned to -135 degrees
- moved R17 14.3 mm to (148.2, 72.1), turned to 180 degrees
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- renumbered R17 to R15, R18 to R16, R19 to R17
Connections:
- R1 pad 1: /STM32/USART2_TX -> /STM32/USART1_TX
- R2 pad 1: /STM32/USART2_RX -> /STM32/USART1_RX
- R3 pad 1: /STM32/USART1_TX -> /STM32/USART2_TX
- R4 pad 1: /STM32/USART1_RX -> /STM32/USART2_RX
- U4 pad 10: unconnected-(U4-PA0-Pad10) -> STATUS_LED_1
- U4 pad 11: unconnected-(U4-PA1-Pad11) -> STATUS_LED_0
- U4 pad 25: STATUS_LED_0 -> unconnected-(U4-PB12-Pad25)
- U4 pad 26: STATUS_LED_1 -> unconnected-(U4-PB13-Pad26)
Routing:
- net +STM_3V3: track 0.00 -> 185.4 mm, vias 0 -> 9
- net NRST: track 0.00 -> 154.6 mm, vias 0 -> 2
- net BOOT0: track 0.00 -> 148.8 mm, vias 0 -> 2
- net +5V: track 0.00 -> 147.3 mm, vias 0 -> 1
- net /Power/BATTERY_VOLTAGE: track 0.00 -> 114.6 mm, vias 0 -> 2
- net STATUS_LED_1: track 0.00 -> 86.5 mm
- net STATUS_LED_0: track 0.00 -> 75.4 mm
- net /LoRA/AUX: track 0.00 -> 73.3 mm, vias 0 -> 1
- net /STM32/USART2_TX: track 0.00 -> 65.3 mm
- net SYS_JTCK-SWCLK: track 0.00 -> 55.0 mm
- net SYS_JTMS-SWDIO: track 0.00 -> 54.7 mm
- net /STM32/USART2_RX: track 0.00 -> 54.2 mm
- net SYS_JTDO-SWO: track 0.00 -> 46.0 mm
- net +CRYPT_3V3: track 0.00 -> 41.1 mm
- net /LoRA/LORA_M0: track 0.00 -> 39.9 mm
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- added copper zone on F.Cu, net +5V
- added copper zone on B.Cu, net +BATT
- added copper zone on F.Cu, net +VCOM
- added copper zone on B.Cu, net /Power/PMOS_GATE
- added copper zone on F.Cu, net /Power/SW
- added copper zone on B.Cu, net GND
- added copper zone on F.Cu, net GND
- added copper zone on B.Cu, net Net-(D2-K)

Commit message: finished pcb
Parts:
- added G***: LOGO, LOGO, B.Cu at (194.6, 70.8)
- added G***: LOGO, LOGO, B.Cu at (194.6, 94.9)
- added J1: Conn_01x02_Pin, Connector_PinHeader_2.54mm:PinHeader_1x02_P2.54mm_Vertical, F.Cu at (97.8, 62.8)
- added J4: Conn_01x02_Pin, Connector_PinHeader_2.54mm:PinHeader_1x02_P2.54mm_Vertical, F.Cu at (108.7, 120.2)
- added J6: Conn_01x02_Pin, Connector_PinHeader_2.54mm:PinHeader_1x02_P2.54mm_Vertical, F.Cu at (107.6, 62.8)
- added REF**: KiCad-Logo_5mm_SilkScreen, Symbol:KiCad-Logo_5mm_SilkScreen, B.Cu at (99.6, 120.9)
- added TP1: TestPoint, TestPoint:TestPoint_Pad_D1.5mm, F.Cu at (167.6, 97.3)
- added TP2: TestPoint, TestPoint:TestPoint_Pad_D1.5mm, F.Cu at (171.1, 97.3)
- added TP3: TestPoint, TestPoint:TestPoint_Pad_D1.5mm, F.Cu at (174.6, 97.3)
- J3: renamed from J2; footprint Connector_PinHeader_2.54mm:PinHeader_1x06_P2.54mm_Vertical -> Connector_PinHeader_2.54mm:PinHeader_1x06_P2.54mm_Horizontal
- U5, U7: moved to B.Cu
- moved R20 21.6 mm to (117.5, 64.9), turned to 90 degrees
- moved R21 18.4 mm to (120.1, 64.9), turned to 90 degrees
- moved C33 13.9 mm to (114.5, 102.2), turned to 90 degrees
- moved C38 12.9 mm to (123.4, 84.2), turned to -90 degrees
- moved C37 12.8 mm to (125.7, 84.1), turned to -90 degrees
- moved C34 10.1 mm to (116.9, 102.2), turned to 90 degrees
- moved R3 4.90 mm to (124.8, 75.2)
- moved R2 3.23 mm to (125.8, 101.0)
- moved R1 2.19 mm to (125.8, 103.5)
- moved U5 0.61 mm to (103.5, 102.2), turned to 90 degrees
- moved U7 0.14 mm to (103.2, 77.7), turned to 90 degrees
- renumbered J1 to J2
Routing:
- net /GPS/GPS_TX: track 5.60 -> 36.9 mm
- net /GPS/GPS_RX: track 5.60 -> 27.1 mm
- net /LoRA/LORA_TX: track 4.24 -> 24.1 mm
- net /LoRA/LORA_M1: track 39.1 -> 57.5 mm, vias 0 -> 1
- net /LoRA/LORA_RX: track 4.22 -> 20.5 mm
- net /LoRA/LORA_M0: track 39.9 -> 55.5 mm
- net /Crypt/CRYPT_SDA: track 10.4 -> 24.1 mm, vias 0 -> 2
- net +5V: track 147.3 -> 134.4 mm
- net /Crypt/CRYPT_SCL: track 10.5 -> 22.9 mm, vias 0 -> 2
- net /STM32/USART1_RX: track 39.0 -> 45.3 mm
- net /LoRA/AUX: track 73.3 -> 67.5 mm
- net /STM32/USART2_TX: track 65.3 -> 59.7 mm
- net /STM32/USART1_TX: track 38.1 -> 39.8 mm
- net GND: track 0.00 -> 0.03 mm, vias 1199 -> 1154
Other:
- board text added: "+3V3"
- board text added: "BOOT0"
- board text added: "BOOT1"
- board text added: "CRYPT"
- board text added: "CRYPT TEST"
- board text added: "GND"
- board text added: "GND TEST"
- board text added: "GPS NEO - M8N"
- board text added: "GSP TEST"
- board text added: "LED-0"
- board text added: "LED-1"
- board text added: "LORA"
- board text added: "LORA TEST"
- board text added: "NRST"
- board text added: "PROG LED"
- board text added: "RX"
- board text added: "SCL"
- board text added: "SDA"
- board text added: "SWCLK"
- board text added: "SWDIO"
- board text added: "SWITCH <- ON / OFF ->"
- board text added: "SWO"
- board text added: "TAMP"
- board text added: "TX"
- board text added: "USB-C"
- board text added: "{dblquote}SHINZOU SASAGEYO!!{dblquote}"
- board text added: "{dblquote}SIMPLY LOVELY{dblquote}"
