File: hardware/kicad/crypto_node.kicad_pcb (KiCad board)
At the start: 2 copper layers, 129.4 x 65.4 mm, 103 parts, among them J1 Conn_01x02_Pin, J2 USB_C_Receptacle_USB2.0_16P, J3 01x06_Pin, J4 Conn_01x02_Pin, J6 Conn_01x02_Pin, Q1 FDN304PZ, SW1 SW_SPDT_321, U1 TPS563201, U2 TLV74333PDBVR, U3 TLV74333PDBVR, U4 STM32F411CEUx, U5 NEO-M8N, U6 SE050, U7 EBYTE_900T20D, Y1 YSX321SL, Y2 YST310S

Commit message: Final hardware cleanup push (hopefully)
Parts:
- D1: value SLESD5Z5C -> SLESD5B5CU
Routing:
- net GND: vias 1154 -> 1153
