File: hardware/kicad/_restore_backup_2026-08-29T23-32-30-141/Crypt.kicad_sch (KiCad schematic)
At the start: 0 parts

Commit message: GPS and LoRA completed
Changed lines of the file:
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@@
 	(generator "eeschema")
 	(generator_version "10.0")
-	(paper "A5")
+	(paper "A4")
 	(hierarchical_label "CRYPT_SDA"
 		(shape bidirectional)
-		(at 132.08 62.23 0)
+		(at 142.24 86.36 0)
 		(effects
 			(font
@@
 	(hierarchical_label "CRYPT_SCL"
 		(shape input)
-		(at 132.08 68.58 0)
+		(at 142.24 92.71 0)
 		(effects
 			(font
