File: hardware/kicad/_restore_backup_2026-08-29T23-32-30-141/STM32.kicad_sch (KiCad schematic)
At the start: 39 parts, among them J5 01x06_Pin, U5 STM32F411CEUx, Y1 YSX321SL-25MHz, Y2 YXC-Y-26

Commit message: GPS and LoRA completed
Connections:
- no-connect marks 35 -> 13
Changed lines of the file:
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@@
-	)
-	(no_connect
-		(at 166.37 72.39)
 	)
 	(no_connect
 		(at 262.89 76.2)
-	)
-	(no_connect
-		(at 166.37 82.55)
 	)
 	(no_connect
@@
 	)
 	(no_connect
-		(at 166.37 74.93)
-	)
-	(no_connect
-		(at 130.81 72.39)
-	)
-	(no_connect
 		(at 57.15 95.25)
 	)
 	(no_connect
-		(at 130.81 85.09)
-	)
-	(no_connect
-		(at 130.81 97.79)
-	)
-	(no_connect
-		(at 166.37 57.15)
-	)
-	(no_connect
 		(at 29.21 95.25)
-	)
-	(no_connect
-		(at 130.81 118.11)
 	)
 	(no_connect
@@
 	)
 	(no_connect
-		(at 130.81 115.57)
-	)
-	(no_connect
-		(at 166.37 54.61)
-	)
-	(no_connect
-		(at 166.37 69.85)
-	)
-	(no_connect
-		(at 130.81 110.49)
-	)
-	(no_connect
 		(at 81.28 -15.24)
 	)
-	(no_connect
-		(at 130.81 113.03)
-	)
-	(no_connect
-		(at 130.81 100.33)
-	)
-	(no_connect
-		(at 130.81 95.25)
-	)
-	(no_connect
-		(at 130.81 107.95)
-	)
-	(no_connect
-		(at 166.37 67.31)
-	)
-	(no_connect
-		(at 166.37 92.71)
-	)
-	(no_connect
-		(at 130.81 82.55)
-	)
-	(no_connect
-		(at 166.37 64.77)
-	)
-	(no_connect
-		(at 166.37 85.09)
-	)
-	(no_connect
-		(at 130.81 92.71)
-	)
 	(polyline
