File: hardware/kicad/_restore_backup_2026-09-03T22-22-46-445/LoRA.kicad_sch (KiCad schematic)
At the start: 7 parts, among them U8 EBYTE_900T20D

Commit message: Add schematic audit, DESIGN_DECISIONS.md, and interactive website
Connections:
- net LORA_M0 renamed M0
- net LORA_M1 renamed M1
