File: hardware/kicad/_restore_backup_2026-09-03T22-22-46-445/Power.kicad_sch (KiCad schematic)
At the start: 53 parts, among them J19 USB_C_Receptacle_USB2.0_16P, Q1 FDN304PZ, SW1 SW_SPDT_321, U2 TLV74333PDBVR, U3 TLV74333PDBVR, U6 MCP73871-2CC

Commit message: Add schematic audit, DESIGN_DECISIONS.md, and interactive website
Parts:
- added C17, C20: 100nF, symbol Device:C
- added C18, C19: 10μF, symbol Device:C
- added U4: TLV74333PDBVR, Package_TO_SOT_SMD:SOT-23-5_HandSoldering, symbol TLV74333PDBVR:TLV74333PDBVR
Connections:
- net +5V: now also C17.1, C18.1, U4.1 (VIN), U4.3 (EN)
- net GND: now also C17.2, C18.2, C19.2, C20.2, U4.2 (GND)
- new net +GPS_3V3: C19.1, C20.1, U4.5 (OUT)
- no-connect marks 27 -> 29
Other:
- note added: "GPS LDO"
