File: hardware/kicad/_restore_backup_2026-09-03T22-22-46-445/STM32.kicad_sch (KiCad schematic)
At the start: 39 parts, among them J5 01x06_Pin, U5 STM32F411CEUx, Y1 YSX321SL-25MHz, Y2 YXC-Y-26

Commit message: Add schematic audit, DESIGN_DECISIONS.md, and interactive website
Changed lines of the file:
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@@
-		)
-	)
-	(hierarchical_label "LORA_CTRL_M0"
-		(shape output)
-		(at 97.79 119.38 180)
-		(effects
-			(font
-				(size 1.27 1.27)
-			)
-			(justify right)
 		)
 	)
@@
 		)
 	)
-	(hierarchical_label "LORA_CRTL_M1"
-		(shape output)
-		(at 97.79 121.92 180)
-		(effects
-			(font
-				(size 1.27 1.27)
-			)
-			(justify right)
-		)
-	)
